File: RTC.kicad_sch (KiCad schematic)
At the start: 3 parts, among them U6 MCP79412, Y2 32.7680kHz

Commit message: f
Parts:
- removed Y2: 32.7680kHz, Crystal:Crystal_AT310_D3.0mm_L10.0mm_Vertical, symbol Device:Crystal_GND2_Small
- added C19, C20: 15pF, Capacitor_SMD:C_0603_1608Metric_Pad1.08x0.95mm_HandSolder, symbol Device:C
- added Y2: 32.7680kHz, Crystal:Crystal_C38-LF_D3.0mm_L8.0mm_Vertical, symbol Device:Crystal_GND3_Small
Connections:
- net GND: now also C19.1, C20.1, Y2.3
- net X1: now reaches U6.1 (X1)
- net X1: now also C19.2, Y2.1
- net X2: now reaches U6.2 (X2)
- net X2: now also C20.2, Y2.2
- net Li-ion-20mm-cell: now reaches BT2.1 (+), U6.3 (BATT)
Other:
- moved on the sheet: BT2, U6
