File: buck.kicad_sch (KiCad schematic)
At the start: 8 parts, among them U7 DIO6012BCST6

Commit message: f
Connections:
- net inductor_buck: now reaches L1.1, U7.3 (LX)
Changed lines of the file:
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@@
+    (effects (font (size 1.27 1.27)) (justify left bottom))
+  )
+  (label "inductor_buck" (at 119.38 59.69 90)
+    (effects (font (size 1.27 1.27)) (justify left bottom))
+  )
+  (label "buck_output" (at 157.48 59.69 0)
     (effects (font (size 1.27 1.27)) (justify left bottom))
   )
