File: Power.kicad_sch (KiCad schematic)
At the start: 20 parts, among them IC1 AP2112M-3.3TRG1, J3 Conn_01x03, J8 Conn_01x02_Male, J9 USB_B_Mini, Q1 DMG9933USD-13, U5 D1213A-02SM

Commit message: v
Parts:
- added R19: 10k+ pullup, Resistor_SMD:R_0603_1608Metric_Pad0.98x0.95mm_HandSolder, symbol Device:R
Connections:
- net +VDC: now also R19.2; no longer IC1.5 (EN)
- new net 3v3_enable: IC1.5 (EN), R19.1
Other:
- moved on the sheet: C2
Changed lines of the file:
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@@
   (junction (at 87.63 146.05) (diameter 0) (color 0 0 0 0)
   )
+  (junction (at 214.63 53.34) (diameter 0) (color 0 0 0 0)
+  )
   (junction (at 87.63 132.08) (diameter 0) (color 0 0 0 0)
   )
   (junction (at 248.92 121.92) (diameter 0) (color 0 0 0 0)
   )
-  (junction (at 207.01 100.33) (diameter 0) (color 0 0 0 0)
-  )
   (junction (at 80.01 64.77) (diameter 0) (color 0 0 0 0)
   )
@@
   (junction (at 254 121.92) (diameter 0) (color 0 0 0 0)
   )
-  (junction (at 226.314 53.34) (diameter 0) (color 0 0 0 0)
-  )
-  (junction (at 220.98 53.34) (diameter 0) (color 0 0 0 0)
-  )
   (junction (at 232.664 58.42) (diameter 0) (color 0 0 0 0)
   )
@@
   (junction (at 251.46 121.92) (diameter 0) (color 0 0 0 0)
   )
+  (junction (at 226.06 53.34) (diameter 0) (color 0 0 0 0)
+  )
   (junction (at 50.165 132.08) (diameter 0) (color 0 0 0 0)
   )
   (junction (at 78.74 102.87) (diameter 0) (color 0 0 0 0)
+  )
+  (junction (at 226.06 60.96) (diameter 0) (color 0 0 0 0)
   )
   (no_connect (at 264.414 58.42))
@@
   (no_connect (at 90.17 58.42))
   (no_connect (at 60.325 58.42))
-  (wire (pts (xy 207.01 100.33) (xy 207.01 102.87))
-    (stroke (width 0) (type default) (color 0 0 0 0))
-  )
   (wire (pts (xy 73.66 102.87) (xy 76.2 102.87))
     (stroke (width 0) (type default) (color 0 0 0 0))
@@
     (stroke (width 0) (type default) (color 0 0 0 0))
   )
-  (wire (pts (xy 233.934 60.96) (xy 226.314 60.96))
+  (wire (pts (xy 224.155 60.96) (xy 226.06 60.96))
     (stroke (width 0) (type default) (color 0 0 0 0))
   )
@@
     (stroke (width 0) (type default) (color 0 0 0 0))
   )
-  (wire (pts (xy 220.98 53.34) (xy 226.314 53.34))
+  (wire (pts (xy 214.63 53.34) (xy 226.06 53.34))
     (stroke (width 0) (type default) (color 0 0 0 0))
   )
@@
     (stroke (width 0) (type default) (color 0 0 0 0))
   )
+  (wire (pts (xy 226.06 60.96) (xy 233.934 60.96))
+    (stroke (width 0) (type default) (color 0 0 0 0))
+  )
   (wire (pts (xy 180.34 116.84) (xy 187.96 116.84))
     (stroke (width 0) (type default) (color 0 0 0 0))
@@
     (stroke (width 0) (type default) (color 0 0 0 0))
   )
-  (wire (pts (xy 226.314 53.34) (xy 233.934 53.34))
-    (stroke (width 0) (type default) (color 0 0 0 0))
-  )
   (wire (pts (xy 76.2 128.27) (xy 76.2 146.05))
     (stroke (width 0) (type default) (color 0 0 0 0))
@@
     (stroke (width 0) (type default) (color 0 0 0 0))
   )
-  (wire (pts (xy 210.82 53.34) (xy 220.98 53.34))
+  (wire (pts (xy 210.82 53.34) (xy 214.63 53.34))
     (stroke (width 0) (type default) (color 0 0 0 0))
   )
@@
     (stroke (width 0) (type default) (color 0 0 0 0))
   )
-  (wire (pts (xy 220.98 53.34) (xy 220.98 55.88))
+  (wire (pts (xy 214.63 53.34) (xy 214.63 55.88))
     (stroke (width 0) (type default) (color 0 0 0 0))
   )
@@
     (stroke (width 0) (type default) (color 0 0 0 0))
   )
+  (wire (pts (xy 226.06 53.34) (xy 233.934 53.34))
+    (stroke (width 0) (type default) (color 0 0 0 0))
+  )
   (wire (pts (xy 60.325 53.34) (xy 64.135 53.34))
     (stroke (width 0) (type default) (color 0 0 0 0))
@@
     (stroke (width 0) (type default) (color 0 0 0 0))
   )
-  (wire (pts (xy 220.98 60.96) (xy 220.98 63.5))
+  (wire (pts (xy 214.63 60.96) (xy 214.63 63.5))
     (stroke (width 0) (type default) (color 0 0 0 0))
   )
@@
   )
   (polyline (pts (xy 121.92 95.25) (xy 121.92 144.78))
-    (stroke (width 0) (type default) (color 0 0 0 0))
-  )
-  (wire (pts (xy 226.314 60.96) (xy 226.314 53.34))
     (stroke (width 0) (type default) (color 0 0 0 0))
   )
@@
     )
   )
+  (global_label "3v3_enable" (shape input) (at 224.155 60.96 270) (fields_autoplaced)
+    (effects (font (size 1.27 1.27)) (justify right))
+    (property "Intersheet References" "${INTERSHEET_REFS}" (id 0) (at 224.0756 74.0169 90)
+      (effects (font (size 1.27 1.27)) (justify right) hide)
+    )
+  )
   (global_label "D+" (shape input) (at 99.06 53.34 0) (fields_autoplaced)
     (effects (font (size 1.27 1.27)) (justify left))
@@
     (property "Intersheet References" "${INTERSHEET_REFS}" (id 0) (at 104.3155 55.8006 0)
       (effects (font (size 1.27 1.27)) (justify left) hide)
+    )
+  )
+  (global_label "3v3_enable" (shape input) (at 207.01 102.87 270) (fields_autoplaced)
+    (effects (font (size 1.27 1.27)) (justify right))
+    (property "Intersheet References" "${INTERSHEET_REFS}" (id 0) (at 206.9306 115.9269 90)
+      (effects (font (size 1.27 1.27)) (justify right) hide)
     )
   )
@@
     (pin "1")
   )
+  (symbol (lib_id "Device:R") (at 226.06 57.15 0) (mirror x) (unit 1)
+    (in_bom yes) (on_board yes)
+    (property "Reference" "R19" (id 0) (at 217.805 57.785 90))
+    (property "Value" "10k+ pullup" (id 1) (at 220.345 60.325 90))
+    (property "Footprint" "Resistor_SMD:R_0603_1608Metric_Pad0.98x0.95mm_HandSolder" (id 2) (at 224.282 57.15 90)
+      (effects (font (size 1.27 1.27)) hide)
+    )
+    (property "Datasheet" "~" (id 3) (at 226.06 57.15 0)
+      (effects (font (size 1.27 1.27)) hide)
+    )
+    (pin "1")
+    (pin "2")
+  )
   (symbol (lib_id "power:GND") (at 40.64 135.89 0) (unit 1)
     (in_bom yes) (on_board yes)
@@
     (pin "1")
   )
-  (symbol (lib_id "Device:C_Small") (at 220.98 58.42 0) (unit 1)
-    (in_bom yes) (on_board yes)
-    (property "Reference" "C2" (id 0) (at 215.011 59.69 0)
+  (symbol (lib_id "Device:C_Small") (at 214.63 58.42 0) (unit 1)
+    (in_bom yes) (on_board yes)
+    (property "Reference" "C2" (id 0) (at 208.661 59.69 0)
       (effects (font (size 1.27 1.27)) (justify left))
     )
-    (property "Value" "1u" (id 1) (at 215.011 57.15 0)
+    (property "Value" "1u" (id 1) (at 208.661 57.15 0)
       (effects (font (size 1.27 1.27)) (justify left))
     )
-    (property "Footprint" "Capacitor_SMD:C_0805_2012Metric_Pad1.18x1.45mm_HandSolder" (id 2) (at 220.98 58.42 0)
-      (effects (font (size 1.27 1.27)) hide)
-    )
-    (property "Datasheet" "~" (id 3) (at 220.98 58.42 0)
+    (property "Footprint" "Capacitor_SMD:C_0805_2012Metric_Pad1.18x1.45mm_HandSolder" (id 2) (at 214.63 58.42 0)
+      (effects (font (size 1.27 1.27)) hide)
+    )
+    (property "Datasheet" "~" (id 3) (at 214.63 58.42 0)
       (effects (font (size 1.27 1.27)) hide)
     )
@@
     (pin "2")
   )
-  (symbol (lib_id "power:GND") (at 220.98 63.5 0) (unit 1)
-    (in_bom yes) (on_board yes) (fields_autoplaced)
-    (property "Reference" "#PWR064" (id 0) (at 220.98 69.85 0)
-      (effects (font (size 1.27 1.27)) hide)
-    )
-    (property "Value" "GND" (id 1) (at 220.98 68.58 0)
-      (effects (font (size 1.27 1.27)) hide)
-    )
-    (property "Footprint" "" (id 2) (at 220.98 63.5 0)
-      (effects (font (size 1.27 1.27)) hide)
-    )
-    (property "Datasheet" "" (id 3) (at 220.98 63.5 0)
-      (effects (font (size 1.27 1.27)) hide)
-    )
+  (symbol (lib_id "power:GND") (at 214.63 63.5 0) (unit 1)
+    (in_bom yes) (on_board yes) (fields_autoplaced)
+    (property "Reference" "#PWR064" (id 0) (at 214.63 69.85 0)
+      (effects (font (size 1.27 1.27)) hide)
+    )
+    (property "Value" "GND" (id 1) (at 214.63 68.58 0)
+      (effects (font (size 1.27 1.27)) hide)
+    )
+    (property "Footprint" "" (id 2) (at 214.63 63.5 0)
+      (effects (font (size 1.27 1.27)) hide)
+    )
+    (property "Datasheet" "" (id 3) (at 214.63 63.5 0)
+      (effects (font (size 1.27 1.27)) hide)
+    )

Commit message: t
Parts:
- removed BT1: Battery, symbol Device:Battery
- removed C2: 1u, Capacitor_SMD:C_0805_2012Metric_Pad1.18x1.45mm_HandSolder, symbol Device:C_Small
- added JP3, JP4: SolderJumper, Jumper:SolderJumper-2_P1.3mm_Bridged_RoundedPad1.0x1.5mm, symbol Jumper:SolderJumper_2_Bridged
- added R20, R21, R22: 10k, Resistor_SMD:R_0603_1608Metric_Pad0.98x0.95mm_HandSolder, symbol Device:R
- added R23: 330, Resistor_SMD:R_0603_1608Metric_Pad0.98x0.95mm_HandSolder, symbol Device:R
- added U3: APX810S05, Package_TO_SOT_SMD:SOT-23, symbol My_custom_lib:APX810S05
- D2: footprint Diode_THT:D_DO-15_P15.24mm_Horizontal -> Diode_THT:D_DO-15_P5.08mm_Vertical_KathodeUp
Connections:
- net +3V3: now also JP4.2 (B); no longer R17.2
- net +BATT: now also U3.3 (Vcc)
- net GND: now also R15.1, R21.1, U3.2 (GND); no longer D4.1 (K)
- net VBUS: now also F1.2, JP3.1 (A), R20.2, R22.1; no longer FB1.2, Q1.2 (G1), R15.2
- net VBUS_RAW: now also FB1.1; no longer F1.1
- net VBUS_RAW2: now also F1.1, FB1.2; no longer F1.2, FB1.1
- net at D4.2 (A): now also JP3.2 (B); no longer R15.1
- new net: R20.1, R22.2, R23.2
- new net: JP4.1 (A), R17.2
- new net: D4.1 (K), R15.2
- new net GPIO24: R21.2, R23.1
- new net batt_protection: Q1.2 (G1), U3.1 (RESET)
Other:
- note added: "Power source switching"
- note added: "active when Vbat is under 3.08V active high"
- moved on the sheet: D4, F1, FB1, R10, R15, S1

Commit message: ver1
Parts:
- removed R20, R22: 10k, Resistor_SMD:R_0603_1608Metric_Pad0.98x0.95mm_HandSolder, symbol Device:R
- added R24: 10k, Resistor_SMD:R_0603_1608Metric_Pad0.98x0.95mm_HandSolder, symbol Device:R
- R15: footprint Resistor_THT:R_Axial_DIN0204_L3.6mm_D1.6mm_P2.54mm_Vertical -> Resistor_THT:R_Axial_DIN0204_L3.6mm_D1.6mm_P5.08mm_Vertical
- R23: value 330 -> 5k6
Connections:
- net GND: now also R24.1
- net VBUS: now also R23.2
- net batt_protection: now also R24.2
Other:
- moved on the sheet: R23
Changed lines of the file:
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@@
   (junction (at 87.63 146.05) (diameter 0) (color 0 0 0 0)
   )
+  (junction (at 76.2 146.05) (diameter 0) (color 0 0 0 0)
+  )
   (junction (at 87.63 132.08) (diameter 0) (color 0 0 0 0)
   )
@@
   (junction (at 59.69 132.08) (diameter 0) (color 0 0 0 0)
   )
-  (junction (at 120.015 58.42) (diameter 0) (color 0 0 0 0)
-  )
   (junction (at 120.015 48.26) (diameter 0) (color 0 0 0 0)
   )
@@
   )
   (junction (at 78.74 102.87) (diameter 0) (color 0 0 0 0)
-  )
-  (junction (at 123.19 48.26) (diameter 0) (color 0 0 0 0)
   )
   (junction (at 226.06 60.96) (diameter 0) (color 0 0 0 0)
@@
   (no_connect (at 90.17 58.42))
   (no_connect (at 60.325 58.42))
-  (wire (pts (xy 123.19 48.26) (xy 123.19 49.53))
-    (stroke (width 0) (type default) (color 0 0 0 0))
-  )
   (wire (pts (xy 73.66 102.87) (xy 76.2 102.87))
     (stroke (width 0) (type default) (color 0 0 0 0))
@@
     (stroke (width 0) (type default) (color 0 0 0 0))
   )
-  (wire (pts (xy 120.015 58.42) (xy 123.19 58.42))
-    (stroke (width 0) (type default) (color 0 0 0 0))
-  )
   (wire (pts (xy 274.574 60.96) (xy 274.574 63.5))
     (stroke (width 0) (type default) (color 0 0 0 0))
   )
-  (wire (pts (xy 123.19 57.15) (xy 123.19 58.42))
+  (wire (pts (xy 76.2 146.05) (xy 76.2 148.59))
     (stroke (width 0) (type default) (color 0 0 0 0))
   )
@@
     (stroke (width 0) (type default) (color 0 0 0 0))
   )
-  (wire (pts (xy 120.015 48.26) (xy 120.015 49.53))
+  (wire (pts (xy 120.015 48.26) (xy 120.015 55.245))
     (stroke (width 0) (type default) (color 0 0 0 0))
   )
@@
     (stroke (width 0) (type default) (color 0 0 0 0))
   )
-  (wire (pts (xy 120.015 57.15) (xy 120.015 58.42))
-    (stroke (width 0) (type default) (color 0 0 0 0))
-  )
   (wire (pts (xy 81.28 128.27) (xy 81.28 146.05))
     (stroke (width 0) (type default) (color 0 0 0 0))
@@
     (stroke (width 0) (type default) (color 0 0 0 0))
   )
-  (wire (pts (xy 120.015 58.42) (xy 120.015 61.595))
-    (stroke (width 0) (type default) (color 0 0 0 0))
-  )
   (wire (pts (xy 262.89 128.27) (xy 265.43 128.27))
     (stroke (width 0) (type default) (color 0 0 0 0))
   )
-  (wire (pts (xy 123.19 48.26) (xy 130.81 48.26))
+  (wire (pts (xy 120.015 48.26) (xy 130.81 48.26))
     (stroke (width 0) (type default) (color 0 0 0 0))
   )
@@
     (stroke (width 0) (type default) (color 0 0 0 0))
   )
-  (wire (pts (xy 120.015 69.215) (xy 120.015 71.12))
+  (wire (pts (xy 120.015 62.865) (xy 120.015 71.12))
     (stroke (width 0) (type default) (color 0 0 0 0))
   )
@@
     (stroke (width 0) (type default) (color 0 0 0 0))
   )
+  (wire (pts (xy 76.2 156.21) (xy 76.2 158.75))
+    (stroke (width 0) (type default) (color 0 0 0 0))
+  )
   (wire (pts (xy 114.935 71.12) (xy 120.015 71.12))
     (stroke (width 0) (type default) (color 0 0 0 0))
@@
     (stroke (width 0) (type default) (color 0 0 0 0))
   )
-  (wire (pts (xy 120.015 48.26) (xy 123.19 48.26))
-    (stroke (width 0) (type default) (color 0 0 0 0))
-  )
   (text "400-500mA+ max power usage of MCU" (at 229.87 139.7 0)
     (effects (font (size 1.27 1.27)) (justify left bottom))
@@
     (effects (font (size 1.27 1.27)) (justify left bottom))
   )
-  (text "active when Vbat is under 3.08V\nactive high" (at 40.005 156.845 0)
+  (text "active when Vbat is under 3.08V\nactive high" (at 35.56 156.21 0)
     (effects (font (size 1.27 1.27)) (justify left bottom))
   )
@@
     (pin "8")
   )
-  (symbol (lib_id "Device:R") (at 120.015 65.405 0) (mirror x) (unit 1)
-    (in_bom yes) (on_board yes)
-    (property "Reference" "R23" (id 0) (at 116.205 64.135 0))
-    (property "Value" "330" (id 1) (at 116.205 66.675 0))
-    (property "Footprint" "Resistor_SMD:R_0603_1608Metric_Pad0.98x0.95mm_HandSolder" (id 2) (at 118.237 65.405 90)
-      (effects (font (size 1.27 1.27)) hide)
-    )
-    (property "Datasheet" "~" (id 3) (at 120.015 65.405 0)
+  (symbol (lib_id "Device:R") (at 120.015 59.055 0) (mirror x) (unit 1)
+    (in_bom yes) (on_board yes)
+    (property "Reference" "R23" (id 0) (at 116.205 57.785 0))
+    (property "Value" "5k6" (id 1) (at 116.205 60.325 0))
+    (property "Footprint" "Resistor_SMD:R_0603_1608Metric_Pad0.98x0.95mm_HandSolder" (id 2) (at 118.237 59.055 90)
+      (effects (font (size 1.27 1.27)) hide)
+    )
+    (property "Datasheet" "~" (id 3) (at 120.015 59.055 0)
+      (effects (font (size 1.27 1.27)) hide)
+    )
+    (pin "1")
+    (pin "2")
+  )
+  (symbol (lib_id "Device:R") (at 76.2 152.4 0) (mirror x) (unit 1)
+    (in_bom yes) (on_board yes)
+    (property "Reference" "R24" (id 0) (at 72.39 151.13 0))
+    (property "Value" "10k" (id 1) (at 72.39 153.67 0))
+    (property "Footprint" "Resistor_SMD:R_0603_1608Metric_Pad0.98x0.95mm_HandSolder" (id 2) (at 74.422 152.4 90)
+      (effects (font (size 1.27 1.27)) hide)
+    )
+    (property "Datasheet" "~" (id 3) (at 76.2 152.4 0)
       (effects (font (size 1.27 1.27)) hide)
     )
@@
     (pin "1")
   )
-  (symbol (lib_id "Device:R") (at 120.015 53.34 0) (mirror x) (unit 1)
-    (in_bom yes) (on_board yes)
-    (property "Reference" "R20" (id 0) (at 116.205 52.07 0))
-    (property "Value" "10k" (id 1) (at 116.205 54.61 0))
-    (property "Footprint" "Resistor_SMD:R_0603_1608Metric_Pad0.98x0.95mm_HandSolder" (id 2) (at 118.237 53.34 90)
-      (effects (font (size 1.27 1.27)) hide)
-    )
-    (property "Datasheet" "~" (id 3) (at 120.015 53.34 0)
-      (effects (font (size 1.27 1.27)) hide)
-    )
-    (pin "1")
-    (pin "2")
-  )
   (symbol (lib_id "Device:R") (at 81.28 152.4 0) (mirror x) (unit 1)
     (in_bom yes) (on_board yes)
-    (property "Reference" "R10" (id 0) (at 77.47 151.13 0))
-    (property "Value" "10k" (id 1) (at 77.47 153.67 0))
+    (property "Reference" "R10" (id 0) (at 86.36 151.13 0))
+    (property "Value" "10k" (id 1) (at 86.36 153.67 0))
     (property "Footprint" "Resistor_SMD:R_0603_1608Metric_Pad0.98x0.95mm_HandSolder" (id 2) (at 79.502 152.4 90)
       (effects (font (size 1.27 1.27)) hide)
     )
     (property "Datasheet" "~" (id 3) (at 81.28 152.4 0)
-      (effects (font (size 1.27 1.27)) hide)
-    )
-    (pin "1")
-    (pin "2")
-  )
-  (symbol (lib_id "Device:R") (at 123.19 53.34 0) (mirror y) (unit 1)
-    (in_bom yes) (on_board yes)
-    (property "Reference" "R22" (id 0) (at 127 54.61 0))
-    (property "Value" "10k" (id 1) (at 127 52.07 0))
-    (property "Footprint" "Resistor_SMD:R_0603_1608Metric_Pad0.98x0.95mm_HandSolder" (id 2) (at 124.968 53.34 90)
-      (effects (font (size 1.27 1.27)) hide)
-    )
-    (property "Datasheet" "~" (id 3) (at 123.19 53.34 0)
       (effects (font (size 1.27 1.27)) hide)
     )
@@
     (property "Reference" "R15" (id 0) (at 125.73 130.81 0))
     (property "Value" "4.7k" (id 1) (at 125.73 133.35 0))
-    (property "Footprint" "Resistor_THT:R_Axial_DIN0204_L3.6mm_D1.6mm_P2.54mm_Vertical" (id 2) (at 127.762 132.08 90)
+    (property "Footprint" "Resistor_THT:R_Axial_DIN0204_L3.6mm_D1.6mm_P5.08mm_Vertical" (id 2) (at 127.762 132.08 90)
       (effects (font (size 1.27 1.27)) hide)
     )
@@
       (effects (font (size 1.27 1.27)) hide)
     )
+    (pin "1")
+  )
+  (symbol (lib_id "power:GND") (at 76.2 158.75 0) (unit 1)
+    (in_bom yes) (on_board yes) (fields_autoplaced)
+    (property "Reference" "#PWR064" (id 0) (at 76.2 165.1 0)
+      (effects (font (size 1.27 1.27)) hide)
+    )
+    (property "Value" "GND" (id 1) (at 76.2 163.83 0)
+      (effects (font (size 1.27 1.27)) hide)
+    )
+    (property "Footprint" "" (id 2) (at 76.2 158.75 0)
+      (effects (font (size 1.27 1.27)) hide)
+    )
+    (property "Datasheet" "" (id 3) (at 76.2 158.75 0)
+      (effects (font (size 1.27 1.27)) hide)
+    )
