File: Power.kicad_sch (KiCad schematic)
At the start: 25 parts, among them IC1 AP2112M-3.3TRG1, J3 Conn_01x03, J8 Conn_01x02_Male, J9 USB_B_Mini, Q1 DMG9933USD-13, U3 APX810S05, U5 D1213A-02SM

Commit message: g
Connections:
- net GND: no longer J9.6 (Shield)
- net custom_led: now reaches D6.2 (A), R18.1
- net led_select: now reaches J3.2 (Pin_2), R18.2
- net 3v3_led-jumper: now reaches JP4.1 (A), R17.2
- net 3v3_led: now reaches D5.2 (A), R17.1
- net vbus_led: now reaches D4.1 (K), R15.2
- net vbus_led-jumper: now reaches D4.2 (A), JP3.2 (B)
- no-connect marks 5 -> 6
Other:
- moved on the sheet: R18
Changed lines of the file:
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@@
   (junction (at 76.2 146.05) (diameter 0) (color 0 0 0 0)
   )
+  (junction (at 129.54 117.475) (diameter 0) (color 0 0 0 0)
+  )
   (junction (at 87.63 132.08) (diameter 0) (color 0 0 0 0)
   )
   (junction (at 260.35 128.27) (diameter 0) (color 0 0 0 0)
   )
-  (junction (at 80.01 64.77) (diameter 0) (color 0 0 0 0)
-  )
   (junction (at 59.69 132.08) (diameter 0) (color 0 0 0 0)
   )
@@
   (junction (at 49.53 132.08) (diameter 0) (color 0 0 0 0)
   )
+  (no_connect (at 80.01 64.77))
   (no_connect (at 264.414 58.42))
   (no_connect (at 264.414 60.96))
@@
     (stroke (width 0) (type default) (color 0 0 0 0))
   )
-  (wire (pts (xy 177.8 115.57) (xy 177.8 119.38))
+  (wire (pts (xy 177.8 115.57) (xy 177.8 120.015))
     (stroke (width 0) (type default) (color 0 0 0 0))
   )
@@
     (stroke (width 0) (type default) (color 0 0 0 0))
   )
-  (wire (pts (xy 82.55 63.5) (xy 82.55 64.77))
+  (wire (pts (xy 82.55 63.5) (xy 82.55 66.04))
     (stroke (width 0) (type default) (color 0 0 0 0))
   )
@@
     (stroke (width 0) (type default) (color 0 0 0 0))
   )
+  (wire (pts (xy 125.73 117.475) (xy 129.54 117.475))
+    (stroke (width 0) (type default) (color 0 0 0 0))
+  )
   (wire (pts (xy 210.82 53.34) (xy 226.06 53.34))
     (stroke (width 0) (type default) (color 0 0 0 0))
@@
     (stroke (width 0) (type default) (color 0 0 0 0))
   )
-  (wire (pts (xy 80.01 64.77) (xy 80.01 66.04))
-    (stroke (width 0) (type default) (color 0 0 0 0))
-  )
   (wire (pts (xy 78.74 102.87) (xy 81.28 102.87))
     (stroke (width 0) (type default) (color 0 0 0 0))
@@
     (stroke (width 0) (type default) (color 0 0 0 0))
   )
-  (wire (pts (xy 82.55 64.77) (xy 80.01 64.77))
-    (stroke (width 0) (type default) (color 0 0 0 0))
-  )
   (wire (pts (xy 87.63 142.24) (xy 87.63 146.05))
     (stroke (width 0) (type default) (color 0 0 0 0))
   )
+  (wire (pts (xy 129.54 117.475) (xy 129.54 119.38))
+    (stroke (width 0) (type default) (color 0 0 0 0))
+  )
   (wire (pts (xy 90.17 48.26) (xy 100.33 48.26))
     (stroke (width 0) (type default) (color 0 0 0 0))
@@
     (stroke (width 0) (type default) (color 0 0 0 0))
   )
-  (wire (pts (xy 177.8 127) (xy 177.8 130.81))
+  (wire (pts (xy 177.8 127.635) (xy 177.8 130.81))
     (stroke (width 0) (type default) (color 0 0 0 0))
   )
@@
     (stroke (width 0) (type default) (color 0 0 0 0))
   )
-  (wire (pts (xy 129.54 115.57) (xy 129.54 119.38))
+  (wire (pts (xy 129.54 115.57) (xy 129.54 117.475))
     (stroke (width 0) (type default) (color 0 0 0 0))
   )
@@
     (effects (font (size 0.5 0.5)) (justify right bottom))
   )
+  (label "led_select" (at 177.8 119.38 0)
+    (effects (font (size 1.27 1.27)) (justify left bottom))
+  )
+  (label "vbus_led-jumper" (at 125.73 117.475 90)
+    (effects (font (size 1.27 1.27)) (justify left bottom))
+  )
+  (label "3v3_led" (at 154.94 129.54 0)
+    (effects (font (size 1.27 1.27)) (justify left bottom))
+  )
+  (label "3v3_led-jumper" (at 154.94 117.475 180)
+    (effects (font (size 1.27 1.27)) (justify right bottom))
+  )
   (label "batt_protection" (at 76.2 145.415 90)
     (effects (font (size 1.27 1.27)) (justify left bottom))
@@
     (effects (font (size 1.27 1.27)) (justify right bottom))
   )
+  (label "custom_led" (at 177.8 129.54 0)
+    (effects (font (size 1.27 1.27)) (justify left bottom))
+  )
   (label "VBUS_RAW" (at 95.25 48.26 180)
     (effects (font (size 0.5 0.5)) (justify right bottom))
   )
   (label "lin_reg" (at 265.43 100.33 0)
+    (effects (font (size 1.27 1.27)) (justify left bottom))
+  )
+  (label "vbus_led" (at 129.54 126.365 0)
     (effects (font (size 1.27 1.27)) (justify left bottom))
   )
@@
     (pin "MH4")
   )
-  (symbol (lib_id "Device:R") (at 177.8 123.19 0) (mirror x) (unit 1)
-    (in_bom yes) (on_board yes)
-    (property "Reference" "R18" (id 0) (at 173.99 121.92 0))
-    (property "Value" "330" (id 1) (at 173.99 124.46 0))
-    (property "Footprint" "Resistor_SMD:R_0603_1608Metric_Pad0.98x0.95mm_HandSolder" (id 2) (at 176.022 123.19 90)
-      (effects (font (size 1.27 1.27)) hide)
-    )
-    (property "Datasheet" "~" (id 3) (at 177.8 123.19 0)
+  (symbol (lib_id "Device:R") (at 177.8 123.825 0) (mirror x) (unit 1)
+    (in_bom yes) (on_board yes)
+    (property "Reference" "R18" (id 0) (at 173.99 122.555 0))
+    (property "Value" "330" (id 1) (at 173.99 125.095 0))
+    (property "Footprint" "Resistor_SMD:R_0603_1608Metric_Pad0.98x0.95mm_HandSolder" (id 2) (at 176.022 123.825 90)
+      (effects (font (size 1.27 1.27)) hide)
+    )
+    (property "Datasheet" "~" (id 3) (at 177.8 123.825 0)
       (effects (font (size 1.27 1.27)) hide)
     )
@@
     (pin "2")
   )
-  (symbol (lib_id "power:GND") (at 80.01 66.04 0) (unit 1)
-    (in_bom yes) (on_board yes)
-    (property "Reference" "#PWR033" (id 0) (at 80.01 72.39 0)
-      (effects (font (size 1.27 1.27)) hide)
-    )
-    (property "Value" "GND" (id 1) (at 80.137 70.4342 0)
-      (effects (font (size 1.27 1.27)) hide)
-    )
-    (property "Footprint" "" (id 2) (at 80.01 66.04 0)
-      (effects (font (size 1.27 1.27)) hide)
-    )
-    (property "Datasheet" "" (id 3) (at 80.01 66.04 0)
-      (effects (font (size 1.27 1.27)) hide)
-    )
+  (symbol (lib_id "power:GND") (at 82.55 66.04 0) (unit 1)
+    (in_bom yes) (on_board yes)
+    (property "Reference" "#PWR033" (id 0) (at 82.55 72.39 0)
+      (effects (font (size 1.27 1.27)) hide)
+    )
+    (property "Value" "GND" (id 1) (at 82.677 70.4342 0)
+      (effects (font (size 1.27 1.27)) hide)
+    )
+    (property "Footprint" "" (id 2) (at 82.55 66.04 0)
+      (effects (font (size 1.27 1.27)) hide)
+    )
+    (property "Datasheet" "" (id 3) (at 82.55 66.04 0)
+      (effects (font (size 1.27 1.27)) hide)
+    )

Commit message: g
Parts:
- added J11: Conn_01x01, Connector_PinSocket_2.54mm:PinSocket_1x01_P2.54mm_Vertical, symbol Connector_Generic:Conn_01x01
Connections:
- net at J9.6 (Shield): now also J11.1 (Pin_1)
- no-connect marks 6 -> 5
Changed lines of the file:
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@@
   (junction (at 59.69 132.08) (diameter 0) (color 0 0 0 0)
   )
+  (junction (at 232.41 60.96) (diameter 0) (color 0 0 0 0)
+  )
   (junction (at 120.015 48.26) (diameter 0) (color 0 0 0 0)
   )
@@
   (junction (at 78.74 102.87) (diameter 0) (color 0 0 0 0)
   )
-  (junction (at 226.06 60.96) (diameter 0) (color 0 0 0 0)
-  )
   (junction (at 49.53 132.08) (diameter 0) (color 0 0 0 0)
   )
-  (no_connect (at 80.01 64.77))
   (no_connect (at 264.414 58.42))
+  (no_connect (at 90.17 58.42))
   (no_connect (at 264.414 60.96))
   (no_connect (at 264.414 55.88))
-  (no_connect (at 90.17 58.42))
   (no_connect (at 60.325 58.42))
+  (wire (pts (xy 232.41 60.96) (xy 233.934 60.96))
+    (stroke (width 0) (type default) (color 0 0 0 0))
+  )
   (wire (pts (xy 73.66 102.87) (xy 76.2 102.87))
     (stroke (width 0) (type default) (color 0 0 0 0))
@@
     (stroke (width 0) (type default) (color 0 0 0 0))
   )
-  (wire (pts (xy 224.155 60.96) (xy 226.06 60.96))
-    (stroke (width 0) (type default) (color 0 0 0 0))
-  )
   (wire (pts (xy 154.94 104.14) (xy 154.94 107.95))
     (stroke (width 0) (type default) (color 0 0 0 0))
@@
     (stroke (width 0) (type default) (color 0 0 0 0))
   )
-  (wire (pts (xy 82.55 63.5) (xy 82.55 66.04))
-    (stroke (width 0) (type default) (color 0 0 0 0))
-  )
   (wire (pts (xy 232.664 55.88) (xy 232.664 58.42))
     (stroke (width 0) (type default) (color 0 0 0 0))
   )
-  (wire (pts (xy 226.06 60.96) (xy 233.934 60.96))
+  (wire (pts (xy 226.06 60.96) (xy 232.41 60.96))
     (stroke (width 0) (type default) (color 0 0 0 0))
   )
@@
     (stroke (width 0) (type default) (color 0 0 0 0))
   )
+  (wire (pts (xy 232.41 60.96) (xy 232.41 63.5))
+    (stroke (width 0) (type default) (color 0 0 0 0))
+  )
   (wire (pts (xy 87.63 142.24) (xy 87.63 146.05))
     (stroke (width 0) (type default) (color 0 0 0 0))
@@
     (stroke (width 0) (type default) (color 0 0 0 0))
   )
+  (wire (pts (xy 78.105 64.77) (xy 80.01 64.77))
+    (stroke (width 0) (type default) (color 0 0 0 0))
+  )
   (wire (pts (xy 90.17 48.26) (xy 100.33 48.26))
     (stroke (width 0) (type default) (color 0 0 0 0))
@@
   )
   (wire (pts (xy 120.015 62.865) (xy 120.015 71.12))
+    (stroke (width 0) (type default) (color 0 0 0 0))
+  )
+  (wire (pts (xy 82.55 63.5) (xy 82.55 69.215))
     (stroke (width 0) (type default) (color 0 0 0 0))
   )
@@
     (effects (font (size 5 5)) (justify left bottom))
   )
-  (text "active high" (at 226.314 63.5 0)
+  (text "active high" (at 242.57 66.04 0)
     (effects (font (size 1.27 1.27)) (justify left bottom))
   )
@@
     )
   )
-  (global_label "3v3_enable" (shape input) (at 224.155 60.96 270) (fields_autoplaced)
+  (global_label "3v3_enable" (shape input) (at 232.41 63.5 270) (fields_autoplaced)
     (effects (font (size 1.27 1.27)) (justify right))
-    (property "Intersheet References" "${INTERSHEET_REFS}" (id 0) (at 224.0756 74.0169 90)
+    (property "Intersheet References" "${INTERSHEET_REFS}" (id 0) (at 232.3306 76.5569 90)
       (effects (font (size 1.27 1.27)) (justify right) hide)
     )
@@
     (pin "2")
   )
-  (symbol (lib_id "power:GND") (at 82.55 66.04 0) (unit 1)
-    (in_bom yes) (on_board yes)
-    (property "Reference" "#PWR033" (id 0) (at 82.55 72.39 0)
-      (effects (font (size 1.27 1.27)) hide)
-    )
-    (property "Value" "GND" (id 1) (at 82.677 70.4342 0)
-      (effects (font (size 1.27 1.27)) hide)
-    )
-    (property "Footprint" "" (id 2) (at 82.55 66.04 0)
-      (effects (font (size 1.27 1.27)) hide)
-    )
-    (property "Datasheet" "" (id 3) (at 82.55 66.04 0)
+  (symbol (lib_id "power:GND") (at 82.55 69.215 0) (unit 1)
+    (in_bom yes) (on_board yes)
+    (property "Reference" "#PWR033" (id 0) (at 82.55 75.565 0)
+      (effects (font (size 1.27 1.27)) hide)
+    )
+    (property "Value" "GND" (id 1) (at 82.677 73.6092 0)
+      (effects (font (size 1.27 1.27)) hide)
+    )
+    (property "Footprint" "" (id 2) (at 82.55 69.215 0)
+      (effects (font (size 1.27 1.27)) hide)
+    )
+    (property "Datasheet" "" (id 3) (at 82.55 69.215 0)
       (effects (font (size 1.27 1.27)) hide)
     )
@@
     (pin "2")
   )
+  (symbol (lib_id "Connector_Generic:Conn_01x01") (at 73.025 64.77 180) (unit 1)
+    (in_bom yes) (on_board yes)
+    (property "Reference" "J11" (id 0) (at 67.945 66.675 0))
+    (property "Value" "Conn_01x01" (id 1) (at 67.945 69.215 0))
+    (property "Footprint" "Connector_PinSocket_2.54mm:PinSocket_1x01_P2.54mm_Vertical" (id 2) (at 73.025 64.77 0)
+      (effects (font (size 1.27 1.27)) hide)
+    )
+    (property "Datasheet" "~" (id 3) (at 73.025 64.77 0)
+      (effects (font (size 1.27 1.27)) hide)
+    )
+    (pin "1")
+  )
   (symbol (lib_id "power:+3.3V") (at 262.89 95.25 0) (unit 1)
