File: Power.kicad_sch (KiCad schematic)
At the start: 26 parts, among them IC1 AP2112M-3.3TRG1, J11 Conn_01x01, J3 Conn_01x03, J8 Conn_01x02_Male, J9 USB_B_Mini, Q1 DMG9933USD-13, U3 APX810S05, U5 D1213A-02SM

Commit message: r
Parts:
- J11, JP3, JP4: now left out of the parts list
Changed lines of the file:
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@@
   )
   (symbol (lib_id "Jumper:SolderJumper_2_Bridged") (at 154.94 111.76 90) (unit 1)
-    (in_bom yes) (on_board yes)
+    (in_bom no) (on_board yes)
     (property "Reference" "JP4" (id 0) (at 147.955 112.395 90)
       (effects (font (size 1.27 1.27)) (justify right))
@@
   )
   (symbol (lib_id "Jumper:SolderJumper_2_Bridged") (at 129.54 111.76 270) (unit 1)
-    (in_bom yes) (on_board yes) (fields_autoplaced)
+    (in_bom no) (on_board yes) (fields_autoplaced)
     (property "Reference" "JP3" (id 0) (at 132.08 110.4899 90)
       (effects (font (size 1.27 1.27)) (justify left))
@@
   )
   (symbol (lib_id "Connector_Generic:Conn_01x01") (at 73.025 64.77 180) (unit 1)
-    (in_bom yes) (on_board yes)
+    (in_bom no) (on_board yes)
     (property "Reference" "J11" (id 0) (at 67.945 66.675 0))
     (property "Value" "Conn_01x01" (id 1) (at 67.945 69.215 0))
