File: RP2040_board1.kicad_sch (KiCad schematic)
At the start: 43 parts, among them J1 Conn_01x02, J10 Conn_01x10, J11 Conn_01x10, J12 Conn_01x10, J2 MEM2051-00-195-00-A, J5 Conn_01x10, SW1 SW_SPST, SW2 SW_SPST, U1 W25Q128JVS, U2 RP2040, U4 DHT11, Y1 ABLS-12.000MHZ-B4-T

Commit message: f
Parts:
- removed J10, J11, J12, J5: Conn_01x10, Connector_PinHeader_2.54mm:PinHeader_1x10_P2.54mm_Vertical, symbol Connector_Generic:Conn_01x10
- added J4, J5: Conn_01x20, Connector_PinSocket_2.54mm:PinSocket_1x20_P2.54mm_Vertical, symbol Connector_Generic:Conn_01x20

Commit message: v
Parts:
- added FID1: Fiducial, Fiducial:Fiducial_0.5mm_Mask1mm, symbol Mechanical:Fiducial
- added FID2: Fiducial, Aesthetics:BREADBOARD_SPACING, symbol Mechanical:Fiducial
- added J6: debug, Connector_PinSocket_2.54mm:PinSocket_1x03_P2.54mm_Vertical, symbol Connector_Generic:Conn_01x03
- J4: value Conn_01x20 -> lefl_side
- J5: value Conn_01x20 -> right_side
Connections:
- net +3V3: now also J5.5 (Pin_5)
- net GND: now also J4.13 (Pin_13), J4.18 (Pin_18), J4.3 (Pin_3), J4.8 (Pin_8), J5.13 (Pin_13), J5.18 (Pin_18), J5.3 (Pin_3), J5.8 (Pin_8), J6.2 (Pin_2)
- net GPIO0: now also J4.1 (Pin_1)
- net GPIO1: now also J4.2 (Pin_2)
- net GPIO10: now also J4.14 (Pin_14)
- net GPIO11: now also J4.15 (Pin_15)
- net GPIO12: now also J4.16 (Pin_16)
- net GPIO13: now also J4.17 (Pin_17)
- net GPIO14: now also J4.19 (Pin_19)
- net GPIO15: now also J4.20 (Pin_20)
- net GPIO16: now also J5.20 (Pin_20)
- net GPIO17: now also J5.19 (Pin_19)
- net GPIO18: now also J5.17 (Pin_17)
- net GPIO19: now also J5.16 (Pin_16)
- net GPIO2: now also J4.4 (Pin_4)
- net GPIO20: now also J5.15 (Pin_15)
- net GPIO21: now also J5.14 (Pin_14)
- net GPIO22: now also J5.12 (Pin_12)
- net GPIO26_ADC0: now also J5.10 (Pin_10)
- net GPIO27_ADC1: now also J5.9 (Pin_9)
- net GPIO28_ADC2: now also J5.7 (Pin_7)
- net GPIO3: now also J4.5 (Pin_5)
- net GPIO4: now also J4.6 (Pin_6)
- net GPIO5: now also J4.7 (Pin_7)
- net GPIO6: now also J4.9 (Pin_9)
- net GPIO7: now also J4.10 (Pin_10)
- net GPIO8: now also J4.11 (Pin_11)
- net GPIO9: now also J4.12 (Pin_12)
- net RUN: now also J5.11 (Pin_11)
- net SWCLK: now also J6.1 (Pin_1)
- net SWD: now also J6.3 (Pin_3)
- net VBUS: now also J5.1 (Pin_1)
- net +VDC: now reaches J5.2 (Pin_2)
- net 3v3_enable: now reaches J5.4 (Pin_4)
- no-connect marks 0 -> 1
Other:
- note added: "Fiducial+grafics+orientation"
- note added: "Same as Rpi Zero board on the upper side but with some extrapins on the power side ADC_ref is floating powering from VSYS lower then 3v3 may not work since i only implemented a buck not a boost-buck (chip shortage 2022)"
- note added: "buck boost more stuff"
- note added: "ground this for shutdown"
- note added: "led pin"
- note added: "some fet stuff"
- moved on the sheet: J4, J5

Commit message: t
Parts:
- added J7: debug, Connector_PinSocket_2.54mm:PinSocket_1x03_P2.54mm_Vertical, symbol Connector_Generic:Conn_01x03
- added JP1, JP2: SolderJumper, Jumper:SolderJumper-2_P1.3mm_Bridged_RoundedPad1.0x1.5mm, symbol Jumper:SolderJumper_2_Bridged
Connections:
- net GND: now also J7.2 (Pin_2)
- net GPIO16: no longer D3.1 (I/O1), J2.P7 (DAT0), R9.1
- net GPIO17: no longer D3.3 (I/O2), J2.P2 (CD/DAT3)
- net GPIO18: no longer D3.6 (I/O4), J2.P5 (CLK), R8.1
- net GPIO19: no longer D3.4 (I/O3), J2.P3 (CMD), R16.1
- net GPIO23: now also J7.1 (Pin_1), JP2.1 (A)
- net GPIO24: no longer R13.1, U4.2 (IO)
- net GPIO29_ADC3: now also J7.3 (Pin_3)
- net MFP: now also JP1.1 (A)
- new net: JP2.2 (B), R13.1, U4.2 (IO)
- new net SPI_CLK: D3.6 (I/O4), J2.P5 (CLK), R8.1
- new net SPI_MISO: D3.1 (I/O1), J2.P7 (DAT0), R9.1
- new net SPI_MOSI: D3.4 (I/O3), J2.P3 (CMD), R16.1
- new net SPI_SS: D3.3 (I/O2), J2.P2 (CD/DAT3)
- new net pin: JP1.2 (B)
Other:
- note added: "1-15MHz usable"
- note added: "50mA absolute max sunk/sourced by IC GPIO The GPIOs on RP2040 have four different output drive strengths, which are nominally called 2, 4, 8 and 12mA modes. These are not hard limits, nor do they mean that they will always be sourcing (or sinking) the selected amount of milliamps"
- note removed: "buck boost more stuff"
- note removed: "led pin"
- note removed: "some fet stuff"
- moved on the sheet: R12, R14

Commit message: ver1
Parts:
- removed FID2: Fiducial, Aesthetics:BREADBOARD_SPACING, symbol Mechanical:Fiducial
- removed J7: debug, Connector_PinSocket_2.54mm:PinSocket_1x03_P2.54mm_Vertical, symbol Connector_Generic:Conn_01x03
- added J10, J7: Conn_01x01, Connector_PinSocket_2.54mm:PinSocket_1x01_P2.54mm_Vertical, symbol Connector_Generic:Conn_01x01
- added R20, R22: 10k, Resistor_SMD:R_0603_1608Metric_Pad0.98x0.95mm_HandSolder, symbol Device:R
- C8: footprint Capacitor_THT:CP_Radial_D5.0mm_P2.00mm -> Capacitor_THT:CP_Radial_D8.0mm_P3.50mm
- D1: footprint LED_THT:LED_D5.0mm -> LED_SMD:LED_0603_1608Metric_Pad1.05x0.95mm_HandSolder
- Y1: footprint Crystal:Crystal_SMD_SeikoEpson_MA505-2Pin_12.7x5.1mm -> Z_mycustom_footprint_lib:ATS120SM
Connections:
- net I2C_CLK is gone; now on net GPIO13: R14.1
- net I2C_SDA is gone; now on net GPIO12: R12.1
- net SPI_CLK is gone; now on net GPIO18: D3.6 (I/O4), J2.P5 (CLK), R8.1
- net SPI_MISO is gone; now on net GPIO20: D3.1 (I/O1), J2.P7 (DAT0), R9.1
- net SPI_MOSI is gone; now on net GPIO19: D3.4 (I/O3), J2.P3 (CMD), R16.1
- net SPI_SS is gone; now on net GPIO21: D3.3 (I/O2), J2.P2 (CD/DAT3)
- net pin is gone; now on net GPIO14: JP1.2 (B)
- net +3V3: now also J10.1 (Pin_1)
- net +VDC: now also R20.2
- net GND: now also R22.1
- net GPIO16: now also J2.P8 (DAT1)
- net GPIO17: now also J2.P1 (DAT2)
- net GPIO20: no longer J2.P8 (DAT1)
- net GPIO21: no longer J2.P1 (DAT2)
- net GPIO23: now also J7.1 (Pin_1)
- net GPIO29_ADC3: now also R20.1, R22.2
Other:
- note added: "I2C 1 used for RTC"
- note added: "SPI 0 used for SD card"

Commit message: silkscreen
Other:
- note added: "Batt measurement"
- moved on the sheet: R20, R22
Changed lines of the file:
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@@
   (junction (at 69.596 245.745) (diameter 0) (color 0 0 0 0)
   )
-  (junction (at 199.39 132.08) (diameter 0) (color 0 0 0 0)
+  (junction (at 251.46 99.06) (diameter 0) (color 0 0 0 0)
   )
   (junction (at 38.1 143.51) (diameter 0) (color 0 0 0 0)
@@
     (stroke (width 0) (type default) (color 0 0 0 0))
   )
-  (wire (pts (xy 199.39 120.65) (xy 199.39 123.19))
+  (wire (pts (xy 251.46 87.63) (xy 251.46 90.17))
     (stroke (width 0) (type default) (color 0 0 0 0))
   )
@@
     (stroke (width 0) (type default) (color 0 0 0 0))
   )
+  (polyline (pts (xy 270.51 73.66) (xy 270.51 116.84))
+    (stroke (width 0) (type default) (color 0 0 0 0))
+  )
   (wire (pts (xy 216.535 213.36) (xy 216.535 211.455))
     (stroke (width 0) (type default) (color 0 0 0 0))
@@
     (stroke (width 0) (type default) (color 0 0 0 0))
   )
-  (wire (pts (xy 199.39 132.08) (xy 199.39 133.35))
+  (wire (pts (xy 251.46 99.06) (xy 251.46 100.33))
     (stroke (width 0) (type default) (color 0 0 0 0))
   )
@@
     (stroke (width 0) (type default) (color 0 0 0 0))
   )
-  (wire (pts (xy 199.39 132.08) (xy 201.93 132.08))
+  (wire (pts (xy 251.46 99.06) (xy 254 99.06))
     (stroke (width 0) (type default) (color 0 0 0 0))
   )
@@
     (stroke (width 0) (type default) (color 0 0 0 0))
   )
+  (polyline (pts (xy 270.51 116.84) (xy 233.68 116.84))
+    (stroke (width 0) (type default) (color 0 0 0 0))
+  )
   (wire (pts (xy 78.105 80.645) (xy 64.135 80.645))
     (stroke (width 0) (type default) (color 0 0 0 0))
@@
     (stroke (width 0) (type default) (color 0 0 0 0))
   )
+  (polyline (pts (xy 233.68 73.66) (xy 270.51 73.66))
+    (stroke (width 0) (type default) (color 0 0 0 0))
+  )
   (wire (pts (xy 340.995 149.225) (xy 360.045 149.225))
     (stroke (width 0) (type default) (color 0 0 0 0))
@@
     (stroke (width 0) (type default) (color 0 0 0 0))
   )
-  (wire (pts (xy 199.39 140.97) (xy 199.39 142.24))
+  (wire (pts (xy 251.46 107.95) (xy 251.46 109.22))
     (stroke (width 0) (type default) (color 0 0 0 0))
   )
@@
     (stroke (width 0) (type default) (color 0 0 0 0))
   )
-  (wire (pts (xy 199.39 130.81) (xy 199.39 132.08))
+  (wire (pts (xy 251.46 97.79) (xy 251.46 99.06))
     (stroke (width 0) (type default) (color 0 0 0 0))
   )
@@
   )
   (wire (pts (xy 316.23 76.2) (xy 320.04 76.2))
+    (stroke (width 0) (type default) (color 0 0 0 0))
+  )
+  (polyline (pts (xy 233.68 116.84) (xy 233.68 73.66))
     (stroke (width 0) (type default) (color 0 0 0 0))
   )
@@
     (effects (font (size 1.27 1.27)) (justify left bottom))
   )
-  (text "OTHER" (at 181.61 210.82 0)
+  (text "OTHER" (at 158.75 209.55 0)
     (effects (font (size 5 5)) (justify left bottom))
   )
@@
     (effects (font (size 1.27 1.27)) (justify left bottom))
   )
+  (text "Batt measurement" (at 241.3 77.47 0)
+    (effects (font (size 1.27 1.27)) (justify left bottom))
+  )
   (label "QSPI_SS" (at 81.28 245.745 0)
     (effects (font (size 1.27 1.27)) (justify left bottom))
@@
     (effects (font (size 1.27 1.27)) (justify right bottom))
   )
-  (label "GPIO29_ADC3" (at 201.93 132.08 0)
+  (label "GPIO29_ADC3" (at 254 99.06 0)
     (effects (font (size 1.27 1.27)) (justify left bottom))
   )
@@
     )
   )
-  (symbol (lib_id "Device:R") (at 199.39 127 0) (mirror x) (unit 1)
-    (in_bom yes) (on_board yes)
-    (property "Reference" "R20" (id 0) (at 195.58 125.73 0))
-    (property "Value" "10k" (id 1) (at 195.58 128.27 0))
-    (property "Footprint" "Resistor_SMD:R_0603_1608Metric_Pad0.98x0.95mm_HandSolder" (id 2) (at 197.612 127 90)
-      (effects (font (size 1.27 1.27)) hide)
-    )
-    (property "Datasheet" "~" (id 3) (at 199.39 127 0)
+  (symbol (lib_id "Device:R") (at 251.46 93.98 0) (mirror x) (unit 1)
+    (in_bom yes) (on_board yes)
+    (property "Reference" "R20" (id 0) (at 247.65 92.71 0))
+    (property "Value" "10k" (id 1) (at 247.65 95.25 0))
+    (property "Footprint" "Resistor_SMD:R_0603_1608Metric_Pad0.98x0.95mm_HandSolder" (id 2) (at 249.682 93.98 90)
+      (effects (font (size 1.27 1.27)) hide)
+    )
+    (property "Datasheet" "~" (id 3) (at 251.46 93.98 0)
       (effects (font (size 1.27 1.27)) hide)
     )
@@
     (pin "2")
   )
-  (symbol (lib_id "power:GND") (at 199.39 142.24 0) (unit 1)
-    (in_bom yes) (on_board yes)
-    (property "Reference" "#PWR070" (id 0) (at 199.39 148.59 0)
-      (effects (font (size 1.27 1.27)) hide)
-    )
-    (property "Value" "GND" (id 1) (at 199.517 146.6342 0)
-      (effects (font (size 1.27 1.27)) hide)
-    )
-    (property "Footprint" "" (id 2) (at 199.39 142.24 0)
-      (effects (font (size 1.27 1.27)) hide)
-    )
-    (property "Datasheet" "" (id 3) (at 199.39 142.24 0)
+  (symbol (lib_id "power:GND") (at 251.46 109.22 0) (unit 1)
+    (in_bom yes) (on_board yes)
+    (property "Reference" "#PWR070" (id 0) (at 251.46 115.57 0)
+      (effects (font (size 1.27 1.27)) hide)
+    )
+    (property "Value" "GND" (id 1) (at 251.587 113.6142 0)
+      (effects (font (size 1.27 1.27)) hide)
+    )
+    (property "Footprint" "" (id 2) (at 251.46 109.22 0)
+      (effects (font (size 1.27 1.27)) hide)
+    )
+    (property "Datasheet" "" (id 3) (at 251.46 109.22 0)
       (effects (font (size 1.27 1.27)) hide)
     )
@@
     (pin "2")
   )
-  (symbol (lib_id "Device:R") (at 199.39 137.16 0) (mirror x) (unit 1)
-    (in_bom yes) (on_board yes)
-    (property "Reference" "R22" (id 0) (at 195.58 135.89 0))
-    (property "Value" "10k" (id 1) (at 195.58 138.43 0))
-    (property "Footprint" "Resistor_SMD:R_0603_1608Metric_Pad0.98x0.95mm_HandSolder" (id 2) (at 197.612 137.16 90)
-      (effects (font (size 1.27 1.27)) hide)
-    )
-    (property "Datasheet" "~" (id 3) (at 199.39 137.16 0)
+  (symbol (lib_id "Device:R") (at 251.46 104.14 0) (mirror x) (unit 1)
+    (in_bom yes) (on_board yes)
+    (property "Reference" "R22" (id 0) (at 247.65 102.87 0))
+    (property "Value" "10k" (id 1) (at 247.65 105.41 0))
+    (property "Footprint" "Resistor_SMD:R_0603_1608Metric_Pad0.98x0.95mm_HandSolder" (id 2) (at 249.682 104.14 90)
+      (effects (font (size 1.27 1.27)) hide)
+    )
+    (property "Datasheet" "~" (id 3) (at 251.46 104.14 0)
       (effects (font (size 1.27 1.27)) hide)
     )
@@
     (pin "1")
   )
-  (symbol (lib_id "power:+VDC") (at 199.39 120.65 0) (unit 1)
+  (symbol (lib_id "power:+VDC") (at 251.46 87.63 0) (unit 1)
     (in_bom yes) (on_board yes) (fields_autoplaced)
-    (property "Reference" "#PWR067" (id 0) (at 199.39 123.19 0)
-      (effects (font (size 1.27 1.27)) hide)
-    )
-    (property "Value" "+VDC" (id 1) (at 199.39 113.03 0))
-    (property "Footprint" "" (id 2) (at 199.39 120.65 0)
-      (effects (font (size 1.27 1.27)) hide)
-    )
-    (property "Datasheet" "" (id 3) (at 199.39 120.65 0)
-      (effects (font (size 1.27 1.27)) hide)
-    )
+    (property "Reference" "#PWR067" (id 0) (at 251.46 90.17 0)
+      (effects (font (size 1.27 1.27)) hide)
+    )
+    (property "Value" "+VDC" (id 1) (at 251.46 80.01 0))
+    (property "Footprint" "" (id 2) (at 251.46 87.63 0)
+      (effects (font (size 1.27 1.27)) hide)
+    )
+    (property "Datasheet" "" (id 3) (at 251.46 87.63 0)
+      (effects (font (size 1.27 1.27)) hide)
+    )
