File: RP2040_board1.kicad_sch (KiCad schematic)
At the start: 49 parts, among them J1 Conn_01x02, J10 Conn_01x01, J2 MEM2051-00-195-00-A, J4 lefl_side, J5 right_side, J6 debug, J7 Conn_01x01, SW1 SW_SPST, SW2 SW_SPST, U1 W25Q128JVS, U2 RP2040, U4 DHT11, Y1 ABLS-12.000MHZ-B4-T

Commit message: v
Parts:
- added H1, H2, H4: MountingHole, MountingHole:MountingHole_3.2mm_M3, symbol Mechanical:MountingHole
Changed lines of the file:
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@@
     (pin "2")
+  )
+  (symbol (lib_id "Mechanical:MountingHole") (at 354.965 238.76 0) (unit 1)
+    (in_bom yes) (on_board yes)
+    (property "Reference" "H4" (id 0) (at 353.695 234.95 0)
+      (effects (font (size 1.27 1.27)) (justify left))
+    )
+    (property "Value" "MountingHole" (id 1) (at 348.615 243.84 0)
+      (effects (font (size 1.27 1.27)) (justify left))
+    )
+    (property "Footprint" "MountingHole:MountingHole_3.2mm_M3" (id 2) (at 354.965 238.76 0)
+      (effects (font (size 1.27 1.27)) hide)
+    )
+    (property "Datasheet" "~" (id 3) (at 354.965 238.76 0)
+      (effects (font (size 1.27 1.27)) hide)
+    )
   )
   (symbol (lib_id "Device:R") (at 156.845 64.135 270) (unit 1)
@@
     )
     (pin "1")
+  )
+  (symbol (lib_id "Mechanical:MountingHole") (at 312.42 238.76 0) (unit 1)
+    (in_bom yes) (on_board yes)
+    (property "Reference" "H1" (id 0) (at 311.15 234.95 0)
+      (effects (font (size 1.27 1.27)) (justify left))
+    )
+    (property "Value" "MountingHole" (id 1) (at 306.07 243.84 0)
+      (effects (font (size 1.27 1.27)) (justify left))
+    )
+    (property "Footprint" "MountingHole:MountingHole_3.2mm_M3" (id 2) (at 312.42 238.76 0)
+      (effects (font (size 1.27 1.27)) hide)
+    )
+    (property "Datasheet" "~" (id 3) (at 312.42 238.76 0)
+      (effects (font (size 1.27 1.27)) hide)
+    )
   )
   (symbol (lib_id "power:GND") (at 307.594 73.66 270) (unit 1)
@@
     (pin "1")
   )
+  (symbol (lib_id "Mechanical:MountingHole") (at 326.39 238.76 0) (unit 1)
+    (in_bom yes) (on_board yes)
+    (property "Reference" "H2" (id 0) (at 325.12 234.95 0)
+      (effects (font (size 1.27 1.27)) (justify left))
+    )
+    (property "Value" "MountingHole" (id 1) (at 320.04 243.84 0)
+      (effects (font (size 1.27 1.27)) (justify left))
+    )
+    (property "Footprint" "MountingHole:MountingHole_3.2mm_M3" (id 2) (at 326.39 238.76 0)
+      (effects (font (size 1.27 1.27)) hide)
+    )
+    (property "Datasheet" "~" (id 3) (at 326.39 238.76 0)
+      (effects (font (size 1.27 1.27)) hide)
+    )
+  )
   (symbol (lib_id "SamacSys_Parts:D5V0P4UR6SO-7") (at 346.075 96.52 0) (unit 1)
     (in_bom yes) (on_board yes) (fields_autoplaced)
@@
       (reference "FID1") (unit 1) (value "Fiducial") (footprint "Fiducial:Fiducial_0.5mm_Mask1mm")
     )
+    (path "/37e25b07-cf59-45fe-844f-5417bc730cd4"
+      (reference "H1") (unit 1) (value "MountingHole") (footprint "MountingHole:MountingHole_3.2mm_M3")
+    )
+    (path "/875836db-e2df-402a-a219-aedbfdd5ffca"
+      (reference "H2") (unit 1) (value "MountingHole") (footprint "MountingHole:MountingHole_3.2mm_M3")
+    )
+    (path "/0b7e7216-d48e-41fc-8bc4-968fd6608f05"
+      (reference "H4") (unit 1) (value "MountingHole") (footprint "MountingHole:MountingHole_3.2mm_M3")
+    )
     (path "/e2aaeb2d-114e-408c-88f1-df515c6dab22/f62dcee8-aa96-4f0b-935f-e8371ea5d6e2"

Commit message: m
Parts:
- added FID2: Fiducial, Symbol:KiCad-Logo2_8mm_SilkScreen, symbol Mechanical:Fiducial
- added FID3: Fiducial, Symbol:OSHW-Logo2_14.6x12mm_SilkScreen, symbol Mechanical:Fiducial
- U1: value W25Q128JVS -> (none); footprint Package_SO:SOIC-8_5.23x5.23mm_P1.27mm -> (none)
Other:
- moved on the sheet: FID1
Changed lines of the file:
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@@
     (pin "1")
   )
-  (symbol (lib_id "Mechanical:Fiducial") (at 286.385 234.315 0) (unit 1)
+  (symbol (lib_id "Mechanical:Fiducial") (at 275.59 232.41 0) (unit 1)
     (in_bom yes) (on_board yes) (fields_autoplaced)
-    (property "Reference" "FID1" (id 0) (at 289.56 233.0449 0)
-      (effects (font (size 1.27 1.27)) (justify left))
-    )
-    (property "Value" "Fiducial" (id 1) (at 289.56 235.5849 0)
-      (effects (font (size 1.27 1.27)) (justify left))
-    )
-    (property "Footprint" "Fiducial:Fiducial_0.5mm_Mask1mm" (id 2) (at 286.385 234.315 0)
-      (effects (font (size 1.27 1.27)) hide)
-    )
-    (property "Datasheet" "~" (id 3) (at 286.385 234.315 0)
+    (property "Reference" "FID1" (id 0) (at 278.765 231.1399 0)
+      (effects (font (size 1.27 1.27)) (justify left))
+    )
+    (property "Value" "Fiducial" (id 1) (at 278.765 233.6799 0)
+      (effects (font (size 1.27 1.27)) (justify left))
+    )
+    (property "Footprint" "Fiducial:Fiducial_0.5mm_Mask1mm" (id 2) (at 275.59 232.41 0)
+      (effects (font (size 1.27 1.27)) hide)
+    )
+    (property "Datasheet" "~" (id 3) (at 275.59 232.41 0)
       (effects (font (size 1.27 1.27)) hide)
     )
@@
     )
     (pin "1")
+  )
+  (symbol (lib_id "Mechanical:Fiducial") (at 275.59 237.49 0) (unit 1)
+    (in_bom yes) (on_board yes) (fields_autoplaced)
+    (property "Reference" "FID2" (id 0) (at 278.765 236.2199 0)
+      (effects (font (size 1.27 1.27)) (justify left))
+    )
+    (property "Value" "Fiducial" (id 1) (at 278.765 238.7599 0)
+      (effects (font (size 1.27 1.27)) (justify left))
+    )
+    (property "Footprint" "Symbol:KiCad-Logo2_8mm_SilkScreen" (id 2) (at 275.59 237.49 0)
+      (effects (font (size 1.27 1.27)) hide)
+    )
+    (property "Datasheet" "~" (id 3) (at 275.59 237.49 0)
+      (effects (font (size 1.27 1.27)) hide)
+    )
   )
   (symbol (lib_id "power:VBUS") (at 347.345 146.685 0) (unit 1)
@@
     (in_bom yes) (on_board yes)
     (property "Reference" "U1" (id 0) (at 96.52 238.125 0))
-    (property "Value" "W25Q128JVS" (id 1) (at 113.03 258.445 0))
-    (property "Footprint" "Package_SO:SOIC-8_5.23x5.23mm_P1.27mm" (id 2) (at 105.41 248.285 0)
+    (property "Value" "" (id 1) (at 113.03 258.445 0))
+    (property "Footprint" "" (id 2) (at 105.41 248.285 0)
       (effects (font (size 1.27 1.27)) hide)
     )
@@
     )
     (pin "1")
+  )
+  (symbol (lib_id "Mechanical:Fiducial") (at 275.59 243.205 0) (unit 1)
+    (in_bom yes) (on_board yes) (fields_autoplaced)
+    (property "Reference" "FID3" (id 0) (at 278.765 241.9349 0)
+      (effects (font (size 1.27 1.27)) (justify left))
+    )
+    (property "Value" "Fiducial" (id 1) (at 278.765 244.4749 0)
+      (effects (font (size 1.27 1.27)) (justify left))
+    )
+    (property "Footprint" "Symbol:OSHW-Logo2_14.6x12mm_SilkScreen" (id 2) (at 275.59 243.205 0)
+      (effects (font (size 1.27 1.27)) hide)
+    )
+    (property "Datasheet" "~" (id 3) (at 275.59 243.205 0)
+      (effects (font (size 1.27 1.27)) hide)
+    )
   )
   (symbol (lib_id "Device:R") (at 223.52 217.17 0) (mirror x) (unit 1)
@@
       (reference "FID1") (unit 1) (value "Fiducial") (footprint "Fiducial:Fiducial_0.5mm_Mask1mm")
     )
+    (path "/1fc1f7a5-2a0c-44bb-8e36-dd6ae1a56c20"
+      (reference "FID2") (unit 1) (value "Fiducial") (footprint "Symbol:KiCad-Logo2_8mm_SilkScreen")
+    )
+    (path "/c127cef7-fbdf-42a7-bf3c-029d6c62a015"
+      (reference "FID3") (unit 1) (value "Fiducial") (footprint "Symbol:OSHW-Logo2_14.6x12mm_SilkScreen")
+    )
     (path "/37e25b07-cf59-45fe-844f-5417bc730cd4"

Commit message: g
Parts:
- U1: value (none) -> W25Q128JVS; footprint (none) -> Package_SO:SOIC-8_5.23x5.23mm_P1.27mm
Connections:
- net GPIO25-led: now reaches D1.2 (A), R6.1
- net XOUT-raw: now reaches R3.2, Y1.2
Changed lines of the file:
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@@
     (stroke (width 0) (type default) (color 0 0 0 0))
   )
-  (wire (pts (xy 296.545 26.797) (xy 296.545 27.94))
+  (wire (pts (xy 296.545 24.13) (xy 296.545 27.94))
     (stroke (width 0) (type default) (color 0 0 0 0))
   )
@@
     (effects (font (size 1.27 1.27)) (justify left bottom))
   )
+  (label "GPIO25-led" (at 24.13 34.29 0)
+    (effects (font (size 1 1)) (justify left bottom))
+  )
   (label "GPIO24" (at 156.845 140.335 180)
     (effects (font (size 1.27 1.27)) (justify right bottom))
@@
     (effects (font (size 1.27 1.27)) (justify left bottom))
   )
+  (label "XOUT-raw" (at 54.61 120.015 180)
+    (effects (font (size 1.27 1.27)) (justify right bottom))
+  )
   (label "USB-" (at 142.875 71.755 0)
     (effects (font (size 1.27 1.27)) (justify left bottom))
@@
   )
   (label "SWCLK" (at 64.135 144.145 0)
-    (effects (font (size 1.27 1.27)) (justify left bottom))
-  )
-  (label "GPIO29_ADC3" (at 318.77 147.32 0)
     (effects (font (size 1.27 1.27)) (justify left bottom))
   )
@@
     (pin "1")
   )
-  (symbol (lib_id "power:+3V3") (at 296.545 26.797 0) (unit 1)
-    (in_bom yes) (on_board yes)
-    (property "Reference" "#PWR027" (id 0) (at 296.545 30.607 0)
-      (effects (font (size 1.27 1.27)) hide)
-    )
-    (property "Value" "+3V3" (id 1) (at 296.545 22.987 0))
-    (property "Footprint" "" (id 2) (at 296.545 26.797 0)
-      (effects (font (size 1.27 1.27)) hide)
-    )
-    (property "Datasheet" "" (id 3) (at 296.545 26.797 0)
+  (symbol (lib_id "power:+3V3") (at 296.545 24.13 0) (unit 1)
+    (in_bom yes) (on_board yes)
+    (property "Reference" "#PWR027" (id 0) (at 296.545 27.94 0)
+      (effects (font (size 1.27 1.27)) hide)
+    )
+    (property "Value" "+3V3" (id 1) (at 296.545 20.32 0))
+    (property "Footprint" "" (id 2) (at 296.545 24.13 0)
+      (effects (font (size 1.27 1.27)) hide)
+    )
+    (property "Datasheet" "" (id 3) (at 296.545 24.13 0)
       (effects (font (size 1.27 1.27)) hide)
     )
@@
     (in_bom yes) (on_board yes)
     (property "Reference" "U1" (id 0) (at 96.52 238.125 0))
-    (property "Value" "" (id 1) (at 113.03 258.445 0))
-    (property "Footprint" "" (id 2) (at 105.41 248.285 0)
+    (property "Value" "W25Q128JVS" (id 1) (at 113.03 258.445 0))
+    (property "Footprint" "Package_SO:SOIC-8_5.23x5.23mm_P1.27mm" (id 2) (at 105.41 248.285 0)
       (effects (font (size 1.27 1.27)) hide)
     )
@@
     )
     (path "/e2aaeb2d-114e-408c-88f1-df515c6dab22/fbb8e0af-da8d-4169-b2a0-386b4e031496/f81df44e-b78a-4cd6-9a03-b053c432e5cb"
-      (reference "RR1") (unit 1) (value "R_Small") (footprint "Resistor_THT:R_Axial_DIN0204_L3.6mm_D1.6mm_P5.08mm_Horizontal")
+      (reference "RR1") (unit 1) (value "R_Small") (footprint "Resistor_THT:R_Axial_DIN0204_L3.6mm_D1.6mm_P5.08mm_Vertical")
     )
     (path "/e2aaeb2d-114e-408c-88f1-df515c6dab22/fbb8e0af-da8d-4169-b2a0-386b4e031496/2982fbde-d7ac-415c-ba98-964a590d7d4e"
-      (reference "RR2") (unit 1) (value "R_Small") (footprint "Resistor_THT:R_Axial_DIN0204_L3.6mm_D1.6mm_P5.08mm_Horizontal")
+      (reference "RR2") (unit 1) (value "R_Small") (footprint "Resistor_THT:R_Axial_DIN0204_L3.6mm_D1.6mm_P5.08mm_Vertical")
     )
     (path "/e2aaeb2d-114e-408c-88f1-df515c6dab22/35a575e5-7e0b-4624-9431-b15d63de581e"

Commit message: g
Parts:
- added H3: MountingHole, MountingHole:MountingHole_3.2mm_M3, symbol Mechanical:MountingHole
Changed lines of the file:
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@@
     (pin "2")
+  )
+  (symbol (lib_id "Mechanical:MountingHole") (at 340.36 238.76 0) (unit 1)
+    (in_bom yes) (on_board yes)
+    (property "Reference" "H3" (id 0) (at 339.09 234.95 0)
+      (effects (font (size 1.27 1.27)) (justify left))
+    )
+    (property "Value" "MountingHole" (id 1) (at 334.01 243.84 0)
+      (effects (font (size 1.27 1.27)) (justify left))
+    )
+    (property "Footprint" "MountingHole:MountingHole_3.2mm_M3" (id 2) (at 340.36 238.76 0)
+      (effects (font (size 1.27 1.27)) hide)
+    )
+    (property "Datasheet" "~" (id 3) (at 340.36 238.76 0)
+      (effects (font (size 1.27 1.27)) hide)
+    )
   )
   (symbol (lib_id "power:GND") (at 105.41 259.715 0) (unit 1)
@@
       (reference "H2") (unit 1) (value "MountingHole") (footprint "MountingHole:MountingHole_3.2mm_M3")
     )
+    (path "/2e02c559-7cf2-4550-8043-f6ed8370edaf"
+      (reference "H3") (unit 1) (value "MountingHole") (footprint "MountingHole:MountingHole_3.2mm_M3")
+    )
     (path "/0b7e7216-d48e-41fc-8bc4-968fd6608f05"
       (reference "H4") (unit 1) (value "MountingHole") (footprint "MountingHole:MountingHole_3.2mm_M3")
@@
       (reference "J10") (unit 1) (value "Conn_01x01") (footprint "Connector_PinSocket_2.54mm:PinSocket_1x01_P2.54mm_Vertical")
     )
+    (path "/e2aaeb2d-114e-408c-88f1-df515c6dab22/d3feea14-ff08-4791-8d7f-466f48bba395"
+      (reference "J11") (unit 1) (value "Conn_01x01") (footprint "Connector_PinSocket_2.54mm:PinSocket_1x01_P2.54mm_Vertical")
+    )
     (path "/e8a6fe2b-2fbf-47dc-a43b-ccbee8db7579"
