File: RP2040_board1.kicad_sch (KiCad schematic)
At the start: 55 parts, among them J1 Conn_01x02, J10 Conn_01x01, J2 MEM2051-00-195-00-A, J4 lefl_side, J5 right_side, J6 debug, J7 Conn_01x01, SW1 SW_SPST, SW2 SW_SPST, U1 W25Q128JVS, U2 RP2040, U4 DHT11, Y1 ABLS-12.000MHZ-B4-T

Commit message: r
Parts:
- FID1, FID2, FID3, H1, H2, H3, H4, J10, J7, JP1, JP2: now left out of the parts list
Changed lines of the file:
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@@
   )
   (symbol (lib_id "Mechanical:MountingHole") (at 354.965 238.76 0) (unit 1)
-    (in_bom yes) (on_board yes)
+    (in_bom no) (on_board yes)
     (property "Reference" "H4" (id 0) (at 353.695 234.95 0)
       (effects (font (size 1.27 1.27)) (justify left))
@@
   )
   (symbol (lib_id "Mechanical:Fiducial") (at 275.59 232.41 0) (unit 1)
-    (in_bom yes) (on_board yes) (fields_autoplaced)
+    (in_bom no) (on_board yes) (fields_autoplaced)
     (property "Reference" "FID1" (id 0) (at 278.765 231.1399 0)
       (effects (font (size 1.27 1.27)) (justify left))
@@
   )
   (symbol (lib_id "Mechanical:Fiducial") (at 275.59 237.49 0) (unit 1)
-    (in_bom yes) (on_board yes) (fields_autoplaced)
+    (in_bom no) (on_board yes) (fields_autoplaced)
     (property "Reference" "FID2" (id 0) (at 278.765 236.2199 0)
       (effects (font (size 1.27 1.27)) (justify left))
@@
   )
   (symbol (lib_id "Mechanical:MountingHole") (at 340.36 238.76 0) (unit 1)
-    (in_bom yes) (on_board yes)
+    (in_bom no) (on_board yes)
     (property "Reference" "H3" (id 0) (at 339.09 234.95 0)
       (effects (font (size 1.27 1.27)) (justify left))
@@
   )
   (symbol (lib_id "Mechanical:MountingHole") (at 312.42 238.76 0) (unit 1)
-    (in_bom yes) (on_board yes)
+    (in_bom no) (on_board yes)
     (property "Reference" "H1" (id 0) (at 311.15 234.95 0)
       (effects (font (size 1.27 1.27)) (justify left))
@@
   )
   (symbol (lib_id "Connector_Generic:Conn_01x01") (at 293.37 204.47 0) (unit 1)
-    (in_bom yes) (on_board yes) (fields_autoplaced)
+    (in_bom no) (on_board yes) (fields_autoplaced)
     (property "Reference" "J10" (id 0) (at 295.91 203.1999 0)
       (effects (font (size 1.27 1.27)) (justify left))
@@
   )
   (symbol (lib_id "Jumper:SolderJumper_2_Bridged") (at 238.76 264.16 180) (unit 1)
-    (in_bom yes) (on_board yes)
+    (in_bom no) (on_board yes)
     (property "Reference" "JP2" (id 0) (at 239.395 271.145 90)
       (effects (font (size 1.27 1.27)) (justify right))
@@
   )
   (symbol (lib_id "Mechanical:MountingHole") (at 326.39 238.76 0) (unit 1)
-    (in_bom yes) (on_board yes)
+    (in_bom no) (on_board yes)
     (property "Reference" "H2" (id 0) (at 325.12 234.95 0)
       (effects (font (size 1.27 1.27)) (justify left))
@@
   )
   (symbol (lib_id "Mechanical:Fiducial") (at 275.59 243.205 0) (unit 1)
-    (in_bom yes) (on_board yes) (fields_autoplaced)
+    (in_bom no) (on_board yes) (fields_autoplaced)
     (property "Reference" "FID3" (id 0) (at 278.765 241.9349 0)
       (effects (font (size 1.27 1.27)) (justify left))
@@
   )
   (symbol (lib_id "Connector_Generic:Conn_01x01") (at 386.08 189.23 90) (unit 1)
-    (in_bom yes) (on_board yes) (fields_autoplaced)
+    (in_bom no) (on_board yes) (fields_autoplaced)
     (property "Reference" "J7" (id 0) (at 388.62 187.9599 90)
       (effects (font (size 1.27 1.27)) (justify right))
@@
   )
   (symbol (lib_id "Jumper:SolderJumper_2_Bridged") (at 204.47 218.44 90) (unit 1)
-    (in_bom yes) (on_board yes)
+    (in_bom no) (on_board yes)
     (property "Reference" "JP1" (id 0) (at 197.485 219.075 90)
       (effects (font (size 1.27 1.27)) (justify right))
