File: RP2040_board1.kicad_pcb (KiCad board)
At the start: 2 copper layers, 73 parts, among them IC1 AP2112M-3.3TRG1, J1 Conn_01x02, J10 Conn_01x10, J11 Conn_01x10, J12 Conn_01x10, J2 MEM2051-00-195-00-A, J3 Conn_01x03, J5 Conn_01x10, J8 Conn_01x02_Male, J9 USB_B_Mini, Q1 DMG9933USD-13, SW1 SW_SPST, SW2 SW_SPST, U1 W25Q128JVS, U2 RP2040, U4 DHT11, U5 D1213A-02SM, U6 MCP79412, U7 DIO6012BCST6, Y1 ABLS-12.000MHZ-B4-T, Y2 32.7680kHz

Commit message: f
Parts:
- removed J10, J11, J12: Conn_01x10, Connector_PinHeader_2.54mm:PinHeader_1x10_P2.54mm_Vertical
- added ?: , Aesthetics:BREADBOARD_SPACING, F.Cu at (250.2, 70.6)
- added C19: 15pF, Capacitor_SMD:C_0603_1608Metric_Pad1.08x0.95mm_HandSolder, F.Cu at (55.6, 159.6)
- added C20: 15pF, Capacitor_SMD:C_0603_1608Metric_Pad1.08x0.95mm_HandSolder, F.Cu at (49.5, 159.6)
- added J4: Conn_01x20, Connector_PinSocket_2.54mm:PinSocket_1x20_P2.54mm_Vertical, F.Cu at (59.3, 32.5)
- BT2: moved to B.Cu
- J5: value Conn_01x10 -> Conn_01x20; footprint Connector_PinHeader_2.54mm:PinHeader_1x10_P2.54mm_Vertical -> Connector_PinSocket_2.54mm:PinSocket_1x20_P2.54mm_Vertical
- Y2: footprint Crystal:Crystal_AT310_D3.0mm_L10.0mm_Vertical -> Crystal:Crystal_C38-LF_D3.0mm_L8.0mm_Vertical
- moved U7 113.3 mm to (221.2, 27.4)
- moved L1 105.3 mm to (215.9, 28.4), turned to 180 degrees
- moved Y2 97.1 mm to (53.5, 158.9), turned to 180 degrees
- moved R1 90.3 mm to (68.3, 74.6)
- moved BT2 89.1 mm to (58.6, 169.5), turned to 180 degrees
- moved R3 86.2 mm to (72.7, 72.1)
- moved J8 85.2 mm to (131.7, 120.4)
- moved R13 83.8 mm to (68.3, 69.6)
- moved R8 79.2 mm to (73.1, 64.6)
- moved R2 74.3 mm to (77.5, 64.6)
- moved U6 74.1 mm to (51.8, 165.2), turned to -90 degrees
- moved U5 73.9 mm to (137.0, 117.2)
- moved C17 69.7 mm to (68.6, 58.8)
- moved C9 67.1 mm to (78.2, 58.8)
- moved D3 66.5 mm to (100.4, 48.9)
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Connections:
- net /RTC/MFP renamed /MFP
- net Net-(BT2-Pad1) renamed /RTC/Li-ion-20mm-cell
- net Net-(L1-Pad1) renamed /Power/buck/inductor_buck
- net Net-(U6-Pad1) renamed /RTC/X1
- J5 pad 1: /GPIO0 -> unconnected-(J5-Pad1)
- J5 pad 10: /GPIO9 -> unconnected-(J5-Pad10)
- J5 pad 2: /GPIO1 -> unconnected-(J5-Pad2)
- J5 pad 3: /GPIO2 -> unconnected-(J5-Pad3)
- J5 pad 4: /GPIO3 -> unconnected-(J5-Pad4)
- J5 pad 5: /GPIO4 -> unconnected-(J5-Pad5)
- J5 pad 6: /GPIO5 -> unconnected-(J5-Pad6)
- J5 pad 7: /GPIO6 -> unconnected-(J5-Pad7)
- J5 pad 8: /GPIO7 -> unconnected-(J5-Pad8)
- J5 pad 9: /GPIO8 -> unconnected-(J5-Pad9)
- U6 pad 2: Net-(U6-Pad2) -> /RTC/X2
- Y2 pad 2: GND -> /RTC/X2
Routing:
- net /RTC/Li-ion-20mm-cell: track 0.00 -> 34.5 mm
- net GND: track 0.00 -> 27.4 mm, vias 0 -> 3
- net /Power/buck_out: track 0.00 -> 15.4 mm
- net Net-(C24-Pad2): track 0.00 -> 13.4 mm
- net /RTC/X1: track 0.00 -> 5.93 mm
- net /RTC/X2: track 0.00 -> 5.84 mm
- net +VDC: track 0.00 -> 3.04 mm
- net /Power/buck/inductor_buck: track 0.00 -> 2.91 mm

Commit message: v
Parts:
- removed ?: , Aesthetics:BREADBOARD_SPACING
- added FID1: Fiducial, Fiducial:Fiducial_0.5mm_Mask1mm, F.Cu at (335.3, 61.0)
- added FID2: Fiducial, Aesthetics:BREADBOARD_SPACING, F.Cu at (340.4, 81.3)
- added J6: debug, Connector_PinSocket_2.54mm:PinSocket_1x03_P2.54mm_Vertical, F.Cu at (124.5, 63.5)
- added R19: 10k+ pullup, Resistor_SMD:R_0603_1608Metric_Pad0.98x0.95mm_HandSolder, F.Cu at (243.8, 30.5)
- J4: value Conn_01x20 -> lefl_side
- J5: value Conn_01x20 -> right_side
- moved J5 222.4 mm to (281.9, 76.2)
- moved J4 207.0 mm to (261.6, 76.2)
- moved D4 126.7 mm to (239.3, 59.6), turned to -90 degrees
- moved U5 121.1 mm to (244.0, 60.6), turned to 180 degrees
- moved FB1 108.3 mm to (250.4, 64.7), turned to 180 degrees
- moved J9 95.9 mm to (243.8, 53.3), turned to 180 degrees
- moved R15 90.3 mm to (239.4, 62.9), turned to -90 degrees
- moved D3 89.4 mm to (15.9, 19.6), turned to 90 degrees
- moved F1 89.4 mm to (250.4, 60.6)
- moved D6 85.5 mm to (96.0, 146.4), turned to -90 degrees
- moved R18 77.2 mm to (94.5, 146.5), turned to 90 degrees
- moved J2 65.3 mm to (17.8, 8.13)
- moved Q1 51.4 mm to (130.3, 147.1)
- moved J3 51.1 mm to (91.9, 142.7), turned to 90 degrees
- moved R10 41.5 mm to (128.5, 150.9), turned to 180 degrees
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Connections:
- IC1 pad 5: +VDC -> 3v3_enable
- J4 pad 1: unconnected-(J4-Pad1) -> /GPIO0
- J4 pad 10: unconnected-(J4-Pad10) -> /GPIO7
- J4 pad 11: unconnected-(J4-Pad11) -> /GPIO8
- J4 pad 12: unconnected-(J4-Pad12) -> /GPIO9
- J4 pad 13: unconnected-(J4-Pad13) -> GND
- J4 pad 14: unconnected-(J4-Pad14) -> /GPIO10
- J4 pad 15: unconnected-(J4-Pad15) -> /GPIO11
- J4 pad 16: unconnected-(J4-Pad16) -> /GPIO12
- J4 pad 17: unconnected-(J4-Pad17) -> /GPIO13
- J4 pad 18: unconnected-(J4-Pad18) -> GND
- J4 pad 19: unconnected-(J4-Pad19) -> /GPIO14
- J4 pad 2: unconnected-(J4-Pad2) -> /GPIO1
- J4 pad 20: unconnected-(J4-Pad20) -> /GPIO15
- J4 pad 3: unconnected-(J4-Pad3) -> GND
- J4 pad 4: unconnected-(J4-Pad4) -> /GPIO2
- J4 pad 5: unconnected-(J4-Pad5) -> /GPIO3
- J4 pad 6: unconnected-(J4-Pad6) -> /GPIO4
- J4 pad 7: unconnected-(J4-Pad7) -> /GPIO5
- J4 pad 8: unconnected-(J4-Pad8) -> GND
- J4 pad 9: unconnected-(J4-Pad9) -> /GPIO6
- J5 pad 1: unconnected-(J5-Pad1) -> VBUS
- J5 pad 10: unconnected-(J5-Pad10) -> /GPIO26_ADC0
- J5 pad 11: unconnected-(J5-Pad11) -> /RUN
- J5 pad 12: unconnected-(J5-Pad12) -> /GPIO22
- J5 pad 13: unconnected-(J5-Pad13) -> GND
- J5 pad 14: unconnected-(J5-Pad14) -> /GPIO21
- J5 pad 15: unconnected-(J5-Pad15) -> /GPIO20
- J5 pad 16: unconnected-(J5-Pad16) -> /GPIO19
- J5 pad 17: unconnected-(J5-Pad17) -> /GPIO18
- J5 pad 18: unconnected-(J5-Pad18) -> GND
- J5 pad 19: unconnected-(J5-Pad19) -> /GPIO17
- J5 pad 2: unconnected-(J5-Pad2) -> +VDC
- J5 pad 20: unconnected-(J5-Pad20) -> /GPIO16
- J5 pad 3: unconnected-(J5-Pad3) -> GND
- J5 pad 4: unconnected-(J5-Pad4) -> 3v3_enable
- J5 pad 5: unconnected-(J5-Pad5) -> +3V3
- J5 pad 7: unconnected-(J5-Pad7) -> /GPIO28_ADC2
- J5 pad 8: unconnected-(J5-Pad8) -> GND
- J5 pad 9: unconnected-(J5-Pad9) -> /GPIO27_ADC1
- U7 pad 1: +VDC -> 3v3_enable

Commit message: t
Parts:
- removed C2: 1u, Capacitor_SMD:C_0805_2012Metric_Pad1.18x1.45mm_HandSolder
- added J7: debug, Connector_PinSocket_2.54mm:PinSocket_1x03_P2.54mm_Vertical, F.Cu at (30.0, -19.3)
- added JP1: SolderJumper, Jumper:SolderJumper-2_P1.3mm_Bridged_RoundedPad1.0x1.5mm, F.Cu at (38.8, -19.9)
- added JP2: SolderJumper, Jumper:SolderJumper-2_P1.3mm_Bridged_RoundedPad1.0x1.5mm, F.Cu at (34.4, -19.9)
- added JP3: SolderJumper, Jumper:SolderJumper-2_P1.3mm_Bridged_RoundedPad1.0x1.5mm, F.Cu at (217.9, 49.3)
- added JP4: SolderJumper, Jumper:SolderJumper-2_P1.3mm_Bridged_RoundedPad1.0x1.5mm, F.Cu at (15.5, -15.4)
- added R20: 10k, Resistor_SMD:R_0603_1608Metric_Pad0.98x0.95mm_HandSolder, F.Cu at (16.0, -20.4)
- added R21: 10k, Resistor_SMD:R_0603_1608Metric_Pad0.98x0.95mm_HandSolder, F.Cu at (20.4, -20.4)
- added R22: 10k, Resistor_SMD:R_0603_1608Metric_Pad0.98x0.95mm_HandSolder, F.Cu at (11.1, -13.4)
- added R23: 330, Resistor_SMD:R_0603_1608Metric_Pad0.98x0.95mm_HandSolder, F.Cu at (11.1, -15.9)
- added U3: APX810S05, Package_TO_SOT_SMD:SOT-23, F.Cu at (206.2, 43.7)
- D2: footprint Diode_THT:D_DO-15_P15.24mm_Horizontal -> Diode_THT:D_DO-15_P5.08mm_Vertical_KathodeUp
- moved FID1 160.1 mm to (175.3, 55.9)
- moved R18 154.9 mm to (218.2, 53.2), turned to 180 degrees
- moved D6 152.7 mm to (218.2, 54.9), turned to 0 degrees
- moved J3 147.9 mm to (209.4, 53.0)
- moved C1 142.8 mm to (-59.8, 62.4)
- moved C10 142.8 mm to (-53.0, 58.7)
- moved C11 142.8 mm to (-65.7, 73.2)
- moved C12 142.8 mm to (-69.4, 65.4)
- moved C13 142.8 mm to (-53.0, 55.7)
- moved C14 142.8 mm to (-74.2, 65.4)
- moved C15 142.8 mm to (-53.0, 61.7)
- moved C16 142.8 mm to (-64.6, 65.4)
- moved C17 142.8 mm to (-74.2, 62.4)
- moved C21 142.8 mm to (21.2, 95.0)
- moved C4 142.8 mm to (-48.2, 55.7)
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Connections:
- D3 pad 1: /GPIO16 -> /SPI_MISO
- D3 pad 3: /GPIO17 -> /SPI_SS
- D3 pad 4: /GPIO19 -> /SPI_MOSI
- D3 pad 6: /GPIO18 -> /SPI_CLK
- D4 pad 1: GND -> Net-(D4-Pad1)
- D4 pad 2: Net-(D4-Pad2) -> Net-(JP3-Pad2)
- F1 pad 1: /Power/VBUS_RAW -> /Power/VBUS_RAW2
- F1 pad 2: /Power/VBUS_RAW2 -> VBUS
- FB1 pad 1: /Power/VBUS_RAW2 -> /Power/VBUS_RAW
- FB1 pad 2: VBUS -> /Power/VBUS_RAW2
- J2 pad P2: /GPIO17 -> /SPI_SS
- J2 pad P3: /GPIO19 -> /SPI_MOSI
- J2 pad P5: /GPIO18 -> /SPI_CLK
- J2 pad P7: /GPIO16 -> /SPI_MISO
- Q1 pad 2: VBUS -> /Power/batt_protection
- R13 pad 1: /GPIO24 -> Net-(R13-Pad1)
- R15 pad 1: Net-(D4-Pad2) -> GND
- R15 pad 2: VBUS -> Net-(D4-Pad1)
- R16 pad 1: /GPIO19 -> /SPI_MOSI
- R17 pad 2: +3V3 -> Net-(R17-Pad2)
- R8 pad 1: /GPIO18 -> /SPI_CLK
- R9 pad 1: /GPIO16 -> /SPI_MISO
- U2 pad 36: /GPIO24 -> GPIO24
- U4 pad 2: /GPIO24 -> Net-(R13-Pad1)
Routing:
- net +BATT: track 0.00 -> 24.4 mm, vias 0 -> 1
- net GND: track 27.4 -> 48.7 mm, vias 3 -> 4
- net VBUS: track 0.00 -> 18.5 mm
- net +VDC: track 3.04 -> 20.2 mm
- net Net-(C24-Pad2): track 13.4 -> 3.13 mm
- net /Power/VBUS_RAW2: track 0.00 -> 10.2 mm
- net /RTC/Li-ion-20mm-cell: track 34.5 -> 27.0 mm
- net Net-(J3-Pad2): track 0.00 -> 6.16 mm
- net /Power/Drains: track 0.00 -> 3.81 mm
- net /RTC/X1: track 5.93 -> 2.14 mm
- net /Power/VBUS_RAW: track 0.00 -> 3.71 mm
- net /RTC/X2: track 5.84 -> 2.14 mm
- net /Power/batt_protection: track 0.00 -> 3.65 mm
- net /Power/buck/inductor_buck: track 2.91 -> 0.00 mm
- net /Power/buck_out: track 15.4 -> 13.0 mm
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- added copper zone on B.Cu, net GND

Commit message: ver1
Parts:
- removed FID2: Fiducial, Aesthetics:BREADBOARD_SPACING
- added J10: Conn_01x01, Connector_PinSocket_2.54mm:PinSocket_1x01_P2.54mm_Vertical, F.Cu at (128.0, 77.6)
- added R24: 10k, Resistor_SMD:R_0603_1608Metric_Pad0.98x0.95mm_HandSolder, F.Cu at (147.3, 69.4)
- BT2: moved to F.Cu
- C10, C12, C14, C15, C16, C17, C4, C5, C6, C9, R11, R16, R8, R9: moved to B.Cu
- C8: footprint Capacitor_THT:CP_Radial_D5.0mm_P2.00mm -> Capacitor_THT:CP_Radial_D8.0mm_P3.50mm
- D1: footprint LED_THT:LED_D5.0mm -> LED_SMD:LED_0603_1608Metric_Pad1.05x0.95mm_HandSolder
- J7: value debug -> Conn_01x01; footprint Connector_PinSocket_2.54mm:PinSocket_1x03_P2.54mm_Vertical -> Connector_PinSocket_2.54mm:PinSocket_1x01_P2.54mm_Vertical
- R15: footprint Resistor_THT:R_Axial_DIN0204_L3.6mm_D1.6mm_P2.54mm_Vertical -> Resistor_THT:R_Axial_DIN0204_L3.6mm_D1.6mm_P5.08mm_Vertical
- R23: value 330 -> 5k6
- Y1: footprint Crystal:Crystal_SMD_SeikoEpson_MA505-2Pin_12.7x5.1mm -> Z_mycustom_footprint_lib:ATS120SM
- moved D3 225.3 mm to (87.1, 94.0), turned to -90 degrees
- moved R13 217.0 mm to (140.2, 105.4), turned to -90 degrees
- moved U4 203.3 mm to (135.0, 108.6), turned to 180 degrees
- moved R1 201.5 mm to (126.3, 60.7)
- moved C7 196.9 mm to (122.7, 68.9), turned to -90 degrees
- moved SW2 189.2 mm to (128.5, 66.8), turned to 90 degrees
- moved R2 189.1 mm to (123.7, 61.5), turned to 90 degrees
- moved C14 182.4 mm to (108.2, 66.3), turned to 90 degrees
- moved C6 181.1 mm to (111.2, 76.8), turned to -90 degrees
- moved C12 179.8 mm to (110.4, 66.4), turned to 90 degrees
- moved C17 179.6 mm to (104.9, 76.2), turned to -90 degrees
- moved R12 178.0 mm to (102.4, 96.5), turned to 90 degrees
- moved C9 177.1 mm to (112.5, 66.4), turned to 90 degrees
- moved Y1 173.9 mm to (95.5, 70.9), turned to -90 degrees
- moved C5 173.6 mm to (113.7, 70.8)
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Connections:
- D3 pad 1: /SPI_MISO -> /GPIO20
- D3 pad 3: /SPI_SS -> /GPIO21
- D3 pad 4: /SPI_MOSI -> /GPIO19
- D3 pad 6: /SPI_CLK -> /GPIO18
- J2 pad P1: /GPIO21 -> /GPIO17
- J2 pad P2: /SPI_SS -> /GPIO21
- J2 pad P3: /SPI_MOSI -> /GPIO19
- J2 pad P5: /SPI_CLK -> /GPIO18
- J2 pad P7: /SPI_MISO -> /GPIO20
- J2 pad P8: /GPIO20 -> /GPIO16
- JP1 pad 2: /pin -> /GPIO14
- R12 pad 1: /I2C_SDA -> /GPIO12
- R14 pad 1: /I2C_CLK -> /GPIO13
- R16 pad 1: /SPI_MOSI -> /GPIO19
- R20 pad 1: Net-(R20-Pad1) -> /GPIO29_ADC3
- R20 pad 2: VBUS -> +VDC
- R22 pad 1: VBUS -> GND
- R22 pad 2: Net-(R20-Pad1) -> /GPIO29_ADC3
- R23 pad 2: Net-(R20-Pad1) -> VBUS
- R8 pad 1: /SPI_CLK -> /GPIO18
- R9 pad 1: /SPI_MISO -> /GPIO20
- U6 pad 5: /I2C_SDA -> /GPIO12
- U6 pad 6: /I2C_CLK -> /GPIO13
Routing:
- net +3V3: track 0.00 -> 262.7 mm, vias 0 -> 18
- net GND: track 48.7 -> 160.4 mm, vias 4 -> 27
- net /GPIO12: track 0.00 -> 81.6 mm, vias 0 -> 6
- net /GPIO13: track 0.00 -> 77.4 mm, vias 0 -> 6
- net /GPIO16: track 0.00 -> 72.1 mm
- net /GPIO14: track 0.00 -> 70.1 mm, vias 0 -> 6
- net VBUS: track 18.5 -> 76.0 mm, vias 0 -> 3
- net +VDC: track 20.2 -> 76.1 mm, vias 0 -> 2
- net /GPIO17: track 0.00 -> 53.6 mm
- net /GPIO22: track 0.00 -> 53.4 mm, vias 0 -> 5
- net /GPIO18: track 0.00 -> 53.1 mm, vias 0 -> 3
- net 3v3_enable: track 0.00 -> 53.1 mm, vias 0 -> 2
- net /GPIO23: track 0.00 -> 53.1 mm, vias 0 -> 1
- net /GPIO20: track 0.00 -> 49.5 mm, vias 0 -> 2
- net /RUN: track 0.00 -> 48.9 mm, vias 0 -> 6
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- added copper zone on F.Cu, net /Power/buck_out
Other:
- board outline added: 90 x 60 mm

Commit message: u
Routing:
- net GND: track 160.4 -> 188.2 mm
Changed lines of the file:
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@@
   (segment (start 108.19784 65.27766) (end 110.32754 65.27766) (width 0.2) (layer "B.Cu") (net 1))
   (segment (start 100.50944 71.64916) (end 100.50944 72.11224) (width 0.5) (layer "B.Cu") (net 1))
+  (segment (start 114.77254 72.32386) (end 114.77254 70.78556) (width 0.5) (layer "B.Cu") (net 1))
   (segment (start 105.06864 72.56466) (end 105.06864 70.01466) (width 0.5) (layer "B.Cu") (net 1))
   (segment (start 104.3543 73.279) (end 105.06864 72.56466) (width 0.5) (layer "B.Cu") (net 1))
+  (segment (start 113.919 73.1774) (end 114.77254 72.32386) (width 0.5) (layer "B.Cu") (net 1))
   (segment (start 106.31242 65.76026) (end 106.34364 65.72904) (width 0.5) (layer "B.Cu") (net 1))
   (segment (start 101.6762 73.279) (end 104.3543 73.279) (width 0.5) (layer "B.Cu") (net 1))
+  (segment (start 109.69946 72.56466) (end 110.3122 73.1774) (width 0.5) (layer "B.Cu") (net 1))
+  (segment (start 113.501509 75.274509) (end 120.38984 75.274509) (width 0.5) (layer "B.Cu") (net 1))
   (segment (start 107.61864 70.01466) (end 107.61864 72.56466) (width 0.5) (layer "B.Cu") (net 1))
   (segment (start 106.34364 65.72904) (end 106.34364 65.37344) (width 0.5) (layer "B.Cu") (net 1))
+  (segment (start 107.61864 71.28966) (end 109.74526 71.28966) (width 0.5) (layer "B.Cu") (net 1))
+  (segment (start 109.74526 71.28966) (end 110.49 72.0344) (width 0.5) (layer "B.Cu") (net 1))
   (segment (start 107.61864 72.56466) (end 105.06864 72.56466) (width 0.5) (layer "B.Cu") (net 1))
   (segment (start 108.19784 65.27766) (end 112.36734 65.27766) (width 0.2) (layer "B.Cu") (net 1))
@@
   (segment (start 112.36734 65.27766) (end 112.46504 65.37536) (width 0.2) (layer "B.Cu") (net 1))
   (segment (start 89.472606 90.678) (end 89.472606 90.374394) (width 0.2) (layer "B.Cu") (net 1))
+  (segment (start 107.61864 72.56466) (end 109.69946 72.56466) (width 0.5) (layer "B.Cu") (net 1))
+  (segment (start 110.49 72.0344) (end 110.49 72.263) (width 0.5) (layer "B.Cu") (net 1))
   (segment (start 106.34364 65.37344) (end 106.3244 65.3542) (width 0.5) (layer "B.Cu") (net 1))
+  (segment (start 110.49 72.263) (end 113.501509 75.274509) (width 0.5) (layer "B.Cu") (net 1))
   (segment (start 89.472606 90.374394) (end 91.43384 88.41316) (width 0.2) (layer "B.Cu") (net 1))
   (segment (start 110.32754 65.27766) (end 110.40764 65.35776) (width 0.2) (layer "B.Cu") (net 1))
   (segment (start 100.50944 72.11224) (end 101.6762 73.279) (width 0.5) (layer "B.Cu") (net 1))
+  (segment (start 111.633 73.1774) (end 113.919 73.1774) (width 0.5) (layer "B.Cu") (net 1))
+  (segment (start 110.3122 73.1774) (end 113.919 73.1774) (width 0.5) (layer "B.Cu") (net 1))
+  (segment (start 110.49 72.0344) (end 111.633 73.1774) (width 0.5) (layer "B.Cu") (net 1))
   (segment (start 105.06864 70.01466) (end 107.61864 70.01466) (width 0.5) (layer "B.Cu") (net 1))
   (segment (start 106.40094 65.27766) (end 108.19784 65.27766) (width 0.5) (layer "B.Cu") (net 1))

Commit message: silkscreen
Parts:
- added kibuzzard-626E7343: G***, kibuzzard-626E7343, F.Cu at (74.1, 60.4)
- added kibuzzard-626E7343: G***, kibuzzard-626E7343, B.Cu at (74.1, 60.5)
- added kibuzzard-626E75F6: G***, kibuzzard-626E75F6, F.Cu at (76.7, 60.4)
- added kibuzzard-626E75F6: G***, kibuzzard-626E75F6, B.Cu at (76.7, 60.5)
- added kibuzzard-626E7607: G***, kibuzzard-626E7607, F.Cu at (104.7, 60.4)
- added kibuzzard-626E7607: G***, kibuzzard-626E7607, B.Cu at (104.1, 85.3)
- added kibuzzard-626E7607: G***, kibuzzard-626E7607, B.Cu at (92.0, 60.5)
- added kibuzzard-626E7607: G***, kibuzzard-626E7607, B.Cu at (116.6, 85.3)
- added kibuzzard-626E7607: G***, kibuzzard-626E7607, B.Cu at (78.7, 85.3)
- added kibuzzard-626E7607: G***, kibuzzard-626E7607, B.Cu at (104.7, 60.5)
- added kibuzzard-626E7607: G***, kibuzzard-626E7607, B.Cu at (91.4, 85.3)
- added kibuzzard-626E7607: G***, kibuzzard-626E7607, F.Cu at (79.3, 60.4)
- added kibuzzard-626E7607: G***, kibuzzard-626E7607, F.Cu at (92.0, 60.4)
- added kibuzzard-626E7607: G***, kibuzzard-626E7607, F.Cu at (91.4, 85.3)
- added kibuzzard-626E7607: G***, kibuzzard-626E7607, F.Cu at (78.7, 85.3)
- added kibuzzard-626E7607: G***, kibuzzard-626E7607, F.Cu at (104.1, 85.3)
- added kibuzzard-626E7607: G***, kibuzzard-626E7607, F.Cu at (116.6, 85.3)
- added kibuzzard-626E7607: G***, kibuzzard-626E7607, B.Cu at (79.3, 60.5)
- added kibuzzard-626E7607: G***, kibuzzard-626E7607, B.Cu at (117.3, 60.5)
- added kibuzzard-626E760F: G***, kibuzzard-626E760F, F.Cu at (81.7, 60.4)
- added kibuzzard-626E760F: G***, kibuzzard-626E760F, B.Cu at (81.8, 60.5)
- added kibuzzard-626E761A: G***, kibuzzard-626E761A, F.Cu at (84.1, 60.4)
- added kibuzzard-626E761A: G***, kibuzzard-626E761A, B.Cu at (84.2, 60.5)
- added kibuzzard-626E7622: G***, kibuzzard-626E7622, F.Cu at (85.5, 60.4)
- added kibuzzard-626E7622: G***, kibuzzard-626E7622, B.Cu at (85.5, 60.5)
- added kibuzzard-626E7694: G***, kibuzzard-626E7694, F.Cu at (88.8, 60.4)
- added kibuzzard-626E7694: G***, kibuzzard-626E7694, B.Cu at (88.8, 60.5)
- added kibuzzard-626E769F: G***, kibuzzard-626E769F, F.Cu at (94.5, 60.4)
- added kibuzzard-626E769F: G***, kibuzzard-626E769F, B.Cu at (94.5, 60.5)
- added kibuzzard-626E76A5: G***, kibuzzard-626E76A5, F.Cu at (96.9, 60.4)
- added kibuzzard-626E76A5: G***, kibuzzard-626E76A5, B.Cu at (96.9, 60.5)
- added kibuzzard-626E76AE: G***, kibuzzard-626E76AE, F.Cu at (99.5, 60.4)
- added kibuzzard-626E76AE: G***, kibuzzard-626E76AE, B.Cu at (99.5, 60.5)
- added kibuzzard-626E76B5: G***, kibuzzard-626E76B5, F.Cu at (102.1, 60.4)
- added kibuzzard-626E76B5: G***, kibuzzard-626E76B5, B.Cu at (102.1, 60.5)
- added kibuzzard-626E76C0: G***, kibuzzard-626E76C0, F.Cu at (107.1, 60.4)
- added kibuzzard-626E76C0: G***, kibuzzard-626E76C0, B.Cu at (107.1, 60.5)
- added kibuzzard-626E76C6: G***, kibuzzard-626E76C6, F.Cu at (109.4, 60.4)
- added kibuzzard-626E76C6: G***, kibuzzard-626E76C6, B.Cu at (109.4, 60.5)
- added kibuzzard-626E76CD: G***, kibuzzard-626E76CD, F.Cu at (112.2, 60.4)
- added kibuzzard-626E76CD: G***, kibuzzard-626E76CD, B.Cu at (112.2, 60.5)
- added kibuzzard-626E76D2: G***, kibuzzard-626E76D2, F.Cu at (114.3, 60.4)
- added kibuzzard-626E76D2: G***, kibuzzard-626E76D2, B.Cu at (114.3, 60.5)
- added kibuzzard-626E76E0: G***, kibuzzard-626E76E0, F.Cu at (122.4, 60.4)
- added kibuzzard-626E76E0: G***, kibuzzard-626E76E0, B.Cu at (119.9, 60.5)
- added kibuzzard-626E76E7: G***, kibuzzard-626E76E7, F.Cu at (124.9, 57.4)
- added kibuzzard-626E76E7: G***, kibuzzard-626E76E7, B.Cu at (122.4, 60.5)
- added kibuzzard-626E934E: G***, kibuzzard-626E934E, F.Cu at (78.5, 75.7)
- added kibuzzard-626E937A: G***, kibuzzard-626E937A, F.Cu at (131.6, 75.4)
- added kibuzzard-626E9458: G***, kibuzzard-626E9458, F.Cu at (75.7, 107.2)
- added kibuzzard-626E946D: G***, kibuzzard-626E946D, F.Cu at (97.8, 103.1)
- added kibuzzard-626E948F: G***, kibuzzard-626E948F, F.Cu at (129.8, 106.2)
- added kibuzzard-626E94A4: G***, kibuzzard-626E94A4, F.Cu at (135.4, 112.3)
- added kibuzzard-626E9527: G***, kibuzzard-626E9527, F.Cu at (73.4, 85.3)
- added kibuzzard-626E9527: G***, kibuzzard-626E9527, B.Cu at (73.4, 85.3)
- added kibuzzard-626E9537: G***, kibuzzard-626E9537, F.Cu at (76.2, 85.3)
- added kibuzzard-626E9537: G***, kibuzzard-626E9537, B.Cu at (76.2, 85.3)
- added kibuzzard-626E966C: G***, kibuzzard-626E966C, F.Cu at (83.8, 85.3)
- added kibuzzard-626E966C: G***, kibuzzard-626E966C, B.Cu at (83.8, 85.3)
- added kibuzzard-626E9677: G***, kibuzzard-626E9677, F.Cu at (81.3, 85.3)
- added kibuzzard-626E9677: G***, kibuzzard-626E9677, B.Cu at (81.3, 85.3)
- added kibuzzard-626E9683: G***, kibuzzard-626E9683, F.Cu at (86.4, 85.3)
- added kibuzzard-626E9683: G***, kibuzzard-626E9683, B.Cu at (86.4, 85.3)
- added kibuzzard-626E968A: G***, kibuzzard-626E968A, F.Cu at (88.9, 85.3)
- added kibuzzard-626E968A: G***, kibuzzard-626E968A, B.Cu at (88.9, 85.3)
- added kibuzzard-626E9692: G***, kibuzzard-626E9692, F.Cu at (94.0, 85.3)
- added kibuzzard-626E9692: G***, kibuzzard-626E9692, B.Cu at (94.0, 85.3)
- added kibuzzard-626E969D: G***, kibuzzard-626E969D, F.Cu at (99.1, 85.3)
- added kibuzzard-626E969D: G***, kibuzzard-626E969D, B.Cu at (99.1, 85.3)
- added kibuzzard-626E96A8: G***, kibuzzard-626E96A8, F.Cu at (101.6, 85.3)
- added kibuzzard-626E96A8: G***, kibuzzard-626E96A8, B.Cu at (101.6, 85.3)
- added kibuzzard-626E96B6: G***, kibuzzard-626E96B6, F.Cu at (125.5, 77.7)
- added kibuzzard-626E96B6: G***, kibuzzard-626E96B6, F.Cu at (111.5, 85.3)
- added kibuzzard-626E96B6: G***, kibuzzard-626E96B6, B.Cu at (111.5, 85.3)
- added kibuzzard-626E96B6: G***, kibuzzard-626E96B6, B.Cu at (125.5, 77.7)
- added kibuzzard-626E96C2: G***, kibuzzard-626E96C2, F.Cu at (114.3, 92.5)
- added kibuzzard-626E96C2: G***, kibuzzard-626E96C2, B.Cu at (114.3, 82.5)
- added kibuzzard-626E96E0: G***, kibuzzard-626E96E0, F.Cu at (114.0, 90.9)
- added kibuzzard-626E96EE: G***, kibuzzard-626E96EE, F.Cu at (119.4, 85.3)
- added kibuzzard-626E96EE: G***, kibuzzard-626E96EE, B.Cu at (119.4, 85.3)
- added kibuzzard-626E96FC: G***, kibuzzard-626E96FC, F.Cu at (122.2, 84.8)
- added kibuzzard-626E96FC: G***, kibuzzard-626E96FC, B.Cu at (122.2, 84.8)
- added kibuzzard-626E977A: G***, kibuzzard-626E977A, F.Cu at (106.7, 91.4)
- added kibuzzard-626E977A: G***, kibuzzard-626E977A, B.Cu at (106.7, 91.4)
- added kibuzzard-626E98D2: G***, kibuzzard-626E98D2, F.Cu at (96.3, 90.4)
- added kibuzzard-626E98D2: G***, kibuzzard-626E98D2, B.Cu at (96.3, 90.4)
Routing:
- net +VDC: track 76.1 -> 77.8 mm
- net /RUN: track 48.9 -> 49.8 mm

Commit message: v
Parts:
- added kibuzzard-626E9458: G***, kibuzzard-626E9458, B.Cu at (80.9, 107.1)
- added kibuzzard-626ED31B: G***, kibuzzard-626ED31B, F.Cu at (74.2, 71.8)
- added kibuzzard-626ED31B: G***, kibuzzard-626ED31B, B.Cu at (74.2, 71.8)
- added kibuzzard-626ED354: G***, kibuzzard-626ED354, F.Cu at (78.3, 62.9)
- added kibuzzard-626ED354: G***, kibuzzard-626ED354, B.Cu at (78.3, 62.9)
- added kibuzzard-626ED41E: G***, kibuzzard-626ED41E, B.Cu at (116.4, 103.9)
- added kibuzzard-626ED435: G***, kibuzzard-626ED435, B.Cu at (150.1, 94.5)
- added kibuzzard-626ED447: G***, kibuzzard-626ED447, B.Cu at (144.5, 73.6)
- added kibuzzard-626ED45F: G***, kibuzzard-626ED45F, B.Cu at (142.7, 68.5)
- moved kibuzzard-626E98D2 1.03 mm to (96.4, 91.4), turned to -90 degrees
- turned kibuzzard-626E7607 to -90 degrees (x3)
- turned kibuzzard-626E7607 to 90 degrees (x3)
- turned kibuzzard-626E76E0 to -90 degrees
- turned kibuzzard-626E76E7 to -90 degrees
