File: RP2040_board1.kicad_pcb (KiCad board)
At the start: 2 copper layers, 90 x 60 mm, 182 parts, among them IC1 AP2112M-3.3TRG1, J1 Conn_01x02, J10 Conn_01x01, J2 MEM2051-00-195-00-A, J3 Conn_01x03, J4 lefl_side, J5 right_side, J6 debug, J7 Conn_01x01, J8 Conn_01x02_Male, J9 USB_B_Mini, Q1 DMG9933USD-13, SW1 SW_SPST, SW2 SW_SPST, U1 W25Q128JVS, U2 RP2040, U3 APX810S05, U4 DHT11, U5 D1213A-02SM, U6 MCP79412, U7 DIO6012BCST6, Y1 ABLS-12.000MHZ-B4-T, Y2 32.7680kHz

Commit message: v
Parts:
- moved R3 2.36 mm to (98.9, 74.3), turned to -90 degrees
- moved R22 1.22 mm to (115.7, 78.8)
- moved R20 1.22 mm to (117.3, 80.7)
- moved C4 1.07 mm to (100.5, 71.6)
- moved C16 0.48 mm to (105.0, 66.3)
Routing:
- net GND: track 188.2 -> 153.5 mm, vias 27 -> 29
- net +1V1: track 9.97 -> 24.3 mm, vias 3 -> 5
- net +3V3: track 262.7 -> 269.4 mm, vias 18 -> 21
- net /RUN: track 49.8 -> 46.1 mm
- net /SWD: track 32.1 -> 35.4 mm
- net /SWCLK: track 36.6 -> 39.8 mm
- net /XOUT: track 2.62 -> 5.53 mm
- net /GPIO29_ADC3: track 11.9 -> 13.0 mm
- net /XIN: track 11.1 -> 10.1 mm
- net Net-(R3-Pad2): track 4.39 -> 3.49 mm
- net /Power/VBUS_RAW: track 3.88 -> 4.70 mm
- net 3v3_enable: track 53.1 -> 52.3 mm
- added copper zone on F.Cu, net +1V1
- added copper zone on F.Cu, net +3V3

Commit message: v
Parts:
- removed kibuzzard-626E934E: G***, kibuzzard-626E934E
- added H1: MountingHole, MountingHole:MountingHole_3.2mm_M3, F.Cu at (76.0, 110.0)
- added H2: MountingHole, MountingHole:MountingHole_3.2mm_M3, F.Cu at (76.0, 80.0)
- added H4: MountingHole, MountingHole:MountingHole_3.2mm_M3, F.Cu at (156.0, 110.0)
- added kibuzzard-6275430A: G***, kibuzzard-6275430A, F.Cu at (78.6, 73.3)
- moved kibuzzard-626E9458 6.02 mm to (78.6, 101.9)
- moved kibuzzard-626E946D 5.29 mm to (103.0, 103.7)
- moved kibuzzard-626ED435 4.57 mm to (151.6, 98.8)
- moved C19 3.86 mm to (98.3, 112.3), turned to 0 degrees
- moved C20 3.83 mm to (101.9, 112.3), turned to 180 degrees
- moved JP1 3.20 mm to (101.0, 93.0)
- moved R9 2.81 mm to (93.0, 104.7)
- moved D3 2.76 mm to (89.8, 93.5)
- moved J2 2.76 mm to (88.3, 105.3)
- moved R11 2.71 mm to (91.8, 109.6), turned to 0 degrees
- moved R8 2.60 mm to (90.7, 104.7)
- moved R16 2.51 mm to (88.6, 104.8)
- moved kibuzzard-626E9458 2.31 mm to (83.2, 107.4)
- moved C11 2.07 mm to (85.6, 94.0)
- moved kibuzzard-626E98D2 0.98 mm to (96.4, 91.4), turned to 90 degrees
Routing:
- net GND: track 153.5 -> 166.3 mm, vias 29 -> 30
- net /GPIO12: track 81.6 -> 76.7 mm, vias 6 -> 8
- net /GPIO18: track 53.1 -> 57.2 mm
- net /GPIO16: track 72.1 -> 70.1 mm
- net +3V3: track 269.4 -> 267.5 mm, vias 21 -> 18
- net /GPIO22: track 53.4 -> 55.2 mm, vias 5 -> 4
- net /GPIO14: track 70.5 -> 72.3 mm
- net /GPIO19: track 48.7 -> 49.9 mm, vias 2 -> 3
- net /GPIO20: track 49.5 -> 50.5 mm
- net /GPIO13: track 76.9 -> 76.2 mm
- net /RTC/X1: track 6.08 -> 6.83 mm
- net +BATT: track 29.3 -> 30.1 mm
- net /RTC/X2: track 6.41 -> 7.15 mm
- net /GPIO17: track 53.6 -> 54.3 mm
- net /MFP: track 7.86 -> 7.18 mm, vias 0 -> 2
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
Commit message: m
Parts:
- added  : LOGO, LOGO, B.Cu at (145.2, 105.5)
- added FID2: Fiducial, Symbol:KiCad-Logo2_8mm_SilkScreen, B.Cu at (83.3, 73.8)
- added FID3: Fiducial, Symbol:OSHW-Logo2_14.6x12mm_SilkScreen, B.Cu at (116.8, 103.8)
- added kibuzzard-627E9976: G***, kibuzzard-627E9976, B.Cu at (155.2, 102.0)
- moved kibuzzard-626ED41E 7.04 mm to (109.3, 104.1)
- moved kibuzzard-626ED435 5.37 mm to (152.3, 93.5)
Routing:
- net +VDC: track 77.4 -> 73.1 mm
- added copper zone on F.Cu, net /Power/buck/inductor_buck

Commit message: g
Routing:
- net +VDC: track 73.1 -> 75.7 mm

Commit message: g
Parts:
- added H3: MountingHole, MountingHole:MountingHole_3.2mm_M3, F.Cu at (156.5, 63.0)
- added J11: Conn_01x01, Connector_PinSocket_2.54mm:PinSocket_1x01_P2.54mm_Vertical, F.Cu at (134.0, 67.1)
- RR1, RR2: footprint Resistor_THT:R_Axial_DIN0204_L3.6mm_D1.6mm_P5.08mm_Horizontal -> Resistor_THT:R_Axial_DIN0204_L3.6mm_D1.6mm_P5.08mm_Vertical
- moved FID1 43.3 mm to (126.5, 92.2), turned to 90 degrees
- moved D2 2.58 mm to (150.6, 69.0)
- moved JP3 1.82 mm to (159.3, 70.9)
- moved kibuzzard-626E96B6 1.53 mm to (125.3, 79.2)
- moved kibuzzard-626E96B6 1.40 mm to (125.3, 79.1)
- moved Q1 0.57 mm to (148.3, 59.7)
- moved R10 0.50 mm to (152.1, 61.8)
- moved J8 0.50 mm to (153.9, 57.2)
Connections:
- net Net-(C24-Pad2) renamed /Power/buck/FB
- net Net-(D1-Pad2) renamed /GPIO25-led
- net Net-(D4-Pad1) renamed /Power/vbus_led
- net Net-(D4-Pad2) renamed /Power/vbus_led-jumper
- net Net-(D5-Pad2) renamed /Power/3v3_led
- net Net-(D6-Pad2) renamed /Power/custom_led
- net Net-(J3-Pad2) renamed /Power/led_select
- net Net-(JP4-Pad1) renamed /Power/3v3_led-jumper
- net Net-(R3-Pad2) renamed /XOUT-raw
- J9 pad 6: GND -> Net-(J9-Pad6)
Routing:
- net GND: track 166.3 -> 191.2 mm, vias 30 -> 48
- net Net-(J9-Pad6): track 0.00 -> 23.3 mm
- net +3V3: track 267.5 -> 275.3 mm
- net VBUS: track 76.5 -> 78.2 mm
- net /Power/vbus_led-jumper: track 3.25 -> 2.37 mm
- net /GPIO18: track 57.2 -> 56.5 mm
- net +VDC: track 75.7 -> 76.3 mm
