File: RP2040_board1.kicad_pcb (KiCad board)
At the start: 2 copper layers, 90 x 60 mm, 191 parts, among them IC1 AP2112M-3.3TRG1, J1 Conn_01x02, J10 Conn_01x01, J11 Conn_01x01, J2 MEM2051-00-195-00-A, J3 Conn_01x03, J4 lefl_side, J5 right_side, J6 debug, J7 Conn_01x01, J8 Conn_01x02_Male, J9 USB_B_Mini, Q1 DMG9933USD-13, SW1 SW_SPST, SW2 SW_SPST, U1 W25Q128JVS, U2 RP2040, U3 APX810S05, U4 DHT11, U5 D1213A-02SM, U6 MCP79412, U7 DIO6012BCST6, Y1 ABLS-12.000MHZ-B4-T, Y2 32.7680kHz

Commit message: f
Other:
- board size 90 x 60 mm -> 90.2 x 60.1 mm
Changed lines of the file:
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@@
     (property "Sheetname" "Power")
     (attr through_hole)
-    (fp_text reference "J8" (at -0.23284 5.08616 90) (layer "F.SilkS")
+    (fp_text reference "J8" (at -1.07104 5.207 180) (layer "F.SilkS")
       (effects (font (size 1 1) (thickness 0.15)))
     )
@@
     (property "Sheetname" "Power")
     (attr exclude_from_pos_files)
-    (fp_text reference "JP3" (at -2.682 0 180) (layer "F.SilkS")
+    (fp_text reference "JP3" (at -2.4534 0 180) (layer "F.SilkS")
       (effects (font (size 1 1) (thickness 0.15)))
     )
@@
     (property "Sheetname" "")
     (attr exclude_from_pos_files)
-    (fp_text reference "H3" (at 3.012 -3.564) (layer "F.SilkS")
+    (fp_text reference "H3" (at 2.885 3.3702) (layer "F.SilkS")
       (effects (font (size 1 1) (thickness 0.15)))
     )
@@
   (gr_line (start 127.254 76.327) (end 126.8095 76.835) (layer "B.SilkS") (width 0.15))
   (gr_rect (start 120.3198 61.9506) (end 120.8278 62.357) (layer "F.SilkS") (width 0.15) (fill solid))
-  (gr_rect (start 71 55) (end 161 115) (layer "Edge.Cuts") (width 0.15) (fill none))
-  (gr_rect (start 71 55) (end 161 115) (layer "Margin") (width 0.15) (fill none))
+  (gr_arc (start 160.994489 111.527352) (mid 160.0454 113.9952) (end 157.603564 115.009339) (layer "Edge.Cuts") (width 0.1))
+  (gr_line (start 157.526752 54.981711) (end 74.171436 54.967461) (layer "Edge.Cuts") (width 0.1))
+  (gr_arc (start 70.780511 58.449448) (mid 71.729601 55.981602) (end 74.171436 54.967461) (layer "Edge.Cuts") (width 0.1))
+  (gr_line (start 70.780511 58.449448) (end 70.766261 111.629564) (layer "Edge.Cuts") (width 0.1))
+  (gr_line (start 74.248248 115.020489) (end 157.603564 115.009339) (layer "Edge.Cuts") (width 0.1))
+  (gr_line (start 160.994489 111.527352) (end 161.008739 58.372636) (layer "Edge.Cuts") (width 0.1))
+  (gr_arc (start 74.248248 115.020489) (mid 71.780372 114.071417) (end 70.766261 111.629564) (layer "Edge.Cuts") (width 0.1))
+  (gr_arc (start 157.526752 54.981711) (mid 159.9946 55.9308) (end 161.008739 58.372636) (layer "Edge.Cuts") (width 0.1))
+  (gr_line (start 70.780332 58.449631) (end 70.766082 111.629747) (layer "Margin") (width 0.1))
+  (gr_arc (start 70.780332 58.449631) (mid 71.729603 55.981955) (end 74.171257 54.967644) (layer "Margin") (width 0.1))
+  (gr_arc (start 157.526935 54.98189) (mid 159.994604 55.931162) (end 161.008922 58.372815) (layer "Margin") (width 0.1))
+  (gr_line (start 74.248069 115.020672) (end 157.603747 115.009518) (layer "Margin") (width 0.1))
+  (gr_arc (start 160.994672 111.527531) (mid 160.0454 113.9952) (end 157.603747 115.009518) (layer "Margin") (width 0.1))
+  (gr_line (start 157.526935 54.98189) (end 74.171257 54.967644) (layer "Margin") (width 0.1))
+  (gr_arc (start 74.248069 115.020672) (mid 71.780403 114.071401) (end 70.766082 111.629747) (layer "Margin") (width 0.1))
+  (gr_line (start 160.994672 111.527531) (end 161.008922 58.372815) (layer "Margin") (width 0.1))
   (dimension (type aligned) (layer "F.Fab")
     (pts (xy 161 55) (xy 71 55))
@@
         (xy 161.544 115.57)
         (xy 70.104 115.57)
-        (xy 70.104 54.61)
-        (xy 161.544 54.61)
+        (xy 70.104 53.2892)
+        (xy 161.544 53.2892)
       )
     )

Commit message: j
Parts:
- added C2: 10u, Capacitor_SMD:C_0805_2012Metric, F.Cu at (136.6, 90.2)
- C18, C3: value 22u -> 10u; footprint Capacitor_THT:CP_Radial_D5.0mm_P2.00mm -> Capacitor_SMD:C_0805_2012Metric
- RR1: value R_Small -> 91k; footprint Resistor_THT:R_Axial_DIN0204_L3.6mm_D1.6mm_P5.08mm_Vertical -> Resistor_SMD:R_0805_2012Metric
- RR2: value R_Small -> 20k; footprint Resistor_THT:R_Axial_DIN0204_L3.6mm_D1.6mm_P5.08mm_Vertical -> Resistor_SMD:R_0805_2012Metric
- moved C18 7.02 mm to (136.6, 86.1), turned to 0 degrees
- moved C3 6.84 mm to (136.6, 88.1), turned to 0 degrees
- moved RR1 6.69 mm to (136.4, 83.3)
- moved RR2 5.40 mm to (134.5, 83.3), turned to 90 degrees
- moved C24 4.93 mm to (138.3, 83.4)
- moved R23 2.33 mm to (135.1, 72.9)
- moved R21 1.12 mm to (136.8, 72.9)
- moved C23 0.77 mm to (135.1, 79.7), turned to 90 degrees
- moved SW2 0.25 mm to (128.3, 66.8)
- moved J11 0.18 mm to (133.8, 67.1)
- moved L1 0.13 mm to (132.0, 88.1), turned to 0 degrees
- moved J3 0.06 mm to (149.1, 77.5)
Routing:
- net VBUS: track 78.2 -> 68.2 mm, vias 3 -> 4
- net GND: track 191.2 -> 199.5 mm, vias 48 -> 53
- net /Power/buck/FB: track 16.8 -> 11.0 mm, vias 2 -> 0
- net 3v3_enable: track 52.3 -> 55.3 mm, vias 2 -> 6
- net /Power/buck_out: track 25.4 -> 23.3 mm
- net +VDC: track 76.3 -> 74.7 mm
- net /Power/buck/inductor_buck: track 2.91 -> 4.34 mm
- net GPIO24: track 43.6 -> 42.4 mm
- net +3V3: track 275.3 -> 275.9 mm, vias 18 -> 16
- added copper zone on F.Cu, net /Power/Drains
- added copper zone on F.Cu, net GND
- removed copper zone on F.Cu, net /Power/buck/inductor_buck
